File: hardware/APRSDongle.sch (KiCad schematic (older format))
At the start: 34 parts, among them IC1 DRA818, J1 SMA, P1 VIN, P2 GPS, P3 PC_CON, P4 CONN_8, P5 SWD, U1 AP7363, U2 KL05

Commit message: finished routing. Gerber generated.
Parts:
- D1: value LED -> PWRSTAT
- renumbered JP2 to DACEN1, C6 to DRAC1, JP3 to DRAPOW1, JP1 to HLSEL1, D3 to STAT0, D4 to STAT1
Changed lines of the file:
@@
 Sheet 1 1
 Title ""
-Date "1 feb 2015"
+Date "2 feb 2015"
 Rev ""
 Comp ""
@@
 $EndComp
 $Comp
-L JUMPER JP2
+L JUMPER DACEN1
 U 1 1 54CD8792
 P 5850 5850
-F 0 "JP2" H 5850 6000 60  0000 C CNN
+F 0 "DACEN1" H 5850 6000 60  0000 C CNN
 F 1 "JUMPER" H 5850 5770 40  0000 C CNN
 F 2 "~" H 5850 5850 60  0000 C CNN
@@
 $EndComp
 $Comp
-L JUMPER JP1
+L JUMPER HLSEL1
 U 1 1 54CD8FA2
 P 5850 5750
-F 0 "JP1" H 5850 5900 60  0000 C CNN
+F 0 "HLSEL1" H 5850 5900 60  0000 C CNN
 F 1 "JUMPER" H 5850 5670 40  0000 C CNN
 F 2 "~" H 5850 5750 60  0000 C CNN
@@
 $EndComp
 $Comp
-L C C6
+L C DRAC1
 U 1 1 54CD92B7
 P 5500 6350
-F 0 "C6" H 5500 6450 40  0000 L CNN
+F 0 "DRAC1" H 5500 6450 40  0000 L CNN
 F 1 "C" H 5506 6265 40  0000 L CNN
 F 2 "~" H 5538 6200 30  0000 C CNN
@@
 	1    0    0    -1
 $EndComp
-Text Label 7550 2250 0    60   ~ 0
+Text Label 7550 2350 0    60   ~ 0
 MC2PC
 Text Label 4950 4200 0    60   ~ 0
@@
 Text Label 5100 3500 0    60   ~ 0
 PC2MC
-Text Label 7550 2350 0    60   ~ 0
+Text Label 7550 2250 0    60   ~ 0
 PC2MC
 $Comp
-L JUMPER JP3
+L JUMPER DRAPOW1
 U 1 1 54CE4DC9
 P 5850 6450
-F 0 "JP3" H 5850 6600 60  0000 C CNN
+F 0 "DRAPOW1" H 5850 6600 60  0000 C CNN
 F 1 "JUMPER" H 5850 6370 40  0000 C CNN
 F 2 "~" H 5850 6450 60  0000 C CNN
@@
 SWD_RST
 $Comp
-L LED D4
+L LED STAT1
 U 1 1 54CE4EFC
 P 3700 2700
-F 0 "D4" H 3700 2800 50  0000 C CNN
+F 0 "STAT1" H 3700 2800 50  0000 C CNN
 F 1 "LED" H 3700 2600 50  0000 C CNN
 F 2 "~" H 3700 2700 60  0000 C CNN
@@
 $EndComp
 $Comp
-L LED D3
+L LED STAT0
 U 1 1 54CE50CC
 P 1900 3500
-F 0 "D3" H 1900 3600 50  0000 C CNN
+F 0 "STAT0" H 1900 3600 50  0000 C CNN
 F 1 "LED" H 1900 3400 50  0000 C CNN
 F 2 "~" H 1900 3500 60  0000 C CNN
@@
 P 950 1450
 F 0 "D1" H 950 1550 50  0000 C CNN
-F 1 "LED" H 950 1350 50  0000 C CNN
+F 1 "PWRSTAT" H 950 1350 50  0000 C CNN
 F 2 "~" H 950 1450 60  0000 C CNN
 F 3 "~" H 950 1450 60  0000 C CNN

Commit message: removed lpf, fixed an error
Parts:
- removed C10, C11: 22p, ~, symbol C
- removed C12, C7: 10p, ~, symbol C
- removed C9: 5p, ~, symbol C
- removed L1: 2Turns, ~, symbol INDUCTOR
- removed L2, L3: 3Turns, ~, symbol INDUCTOR
- renumbered C3 to C1, C4 to C2, C1 to C3, C2 to C4, C8 to C5, C5 to C6, D2 to D1, D1 to D2, R3 to R2, R2 to R3, STAT0 to STAT2
Connections:
- wire segments 111 -> 97
Other:
- note removed: "For this LPF, see \nhttp://www.homingin.com/boxes.html\n"
- moved on the sheet: J1

Commit message: had to fix the netlise.... just dont reanotate. A few more changes, not much
Parts:
- renumbered C3 to C1, C4 to C2, C1 to C3, C2 to C4, C6 to C5, C5 to C8, D2 to D1, D1 to D2, R3 to R2, R2 to R3, STAT2 to STAT0
Changed lines of the file:
@@
 Sheet 1 1
 Title ""
-Date "3 feb 2015"
+Date "4 feb 2015"
 Rev ""
 Comp ""
@@
 ADC0_6
 $Comp
-L C C4
+L C C2
 U 1 1 54CD82EA
 P 1000 4500
-F 0 "C4" H 1000 4600 40  0000 L CNN
+F 0 "C2" H 1000 4600 40  0000 L CNN
 F 1 "100n" H 1006 4415 40  0000 L CNN
 F 2 "~" H 1038 4350 30  0000 C CNN
@@
 $EndComp
 $Comp
-L C C3
+L C C1
 U 1 1 54CD82F9
 P 750 4500
-F 0 "C3" H 750 4600 40  0000 L CNN
+F 0 "C1" H 750 4600 40  0000 L CNN
 F 1 "100n" H 756 4415 40  0000 L CNN
 F 2 "~" H 788 4350 30  0000 C CNN
@@
 DRA2MC
 $Comp
-L C C6
+L C C5
 U 1 1 54CD9232
 P 5050 5850
-F 0 "C6" H 5050 5950 40  0000 L CNN
+F 0 "C5" H 5050 5950 40  0000 L CNN
 F 1 "100u" H 5056 5765 40  0000 L CNN
 F 2 "~" H 5088 5700 30  0000 C CNN
@@
 SQ2MC
 $Comp
-L C C5
+L C C8
 U 1 1 54CE348F
 P 8000 5450
-F 0 "C5" H 8000 5550 40  0000 L CNN
+F 0 "C8" H 8000 5550 40  0000 L CNN
 F 1 "C" H 8006 5365 40  0000 L CNN
 F 2 "~" H 8038 5300 30  0000 C CNN
@@
 $EndComp
 $Comp
-L C C1
+L C C3
 U 1 1 54CE42E1
 P 2050 950
-F 0 "C1" H 2050 1050 40  0000 L CNN
+F 0 "C3" H 2050 1050 40  0000 L CNN
 F 1 "10u" H 2056 865 40  0000 L CNN
 F 2 "~" H 2088 800 30  0000 C CNN
@@
 $EndComp
 $Comp
-L C C2
+L C C4
 U 1 1 54CE4449
 P 3100 950
-F 0 "C2" H 3100 1050 40  0000 L CNN
+F 0 "C4" H 3100 1050 40  0000 L CNN
 F 1 "C" H 3106 865 40  0000 L CNN
 F 2 "~" H 3138 800 30  0000 C CNN
@@
 $EndComp
 $Comp
-L DIODE D1
+L DIODE D2
 U 1 1 54CE4855
 P 1400 700
-F 0 "D1" H 1400 800 40  0000 C CNN
+F 0 "D2" H 1400 800 40  0000 C CNN
 F 1 "DIODE" H 1400 600 40  0000 C CNN
 F 2 "~" H 1400 700 60  0000 C CNN
@@
 $EndComp
 $Comp
-L R R2
+L R R3
 U 1 1 54CE4F0B
 P 3700 2150
-F 0 "R2" V 3780 2150 40  0000 C CNN
+F 0 "R3" V 3780 2150 40  0000 C CNN
 F 1 "R" V 3707 2151 40  0000 C CNN
 F 2 "~" V 3630 2150 30  0000 C CNN
@@
 $EndComp
 $Comp
-L LED STAT2
+L LED STAT0
 U 1 1 54CE50CC
 P 1900 3500
-F 0 "STAT2" H 1900 3600 50  0000 C CNN
+F 0 "STAT0" H 1900 3600 50  0000 C CNN
 F 1 "LED" H 1900 3400 50  0000 C CNN
 F 2 "~" H 1900 3500 60  0000 C CNN
@@
 $EndComp
 $Comp
-L R R3
+L R R2
 U 1 1 54CE50D2
 P 1350 3500
-F 0 "R3" V 1430 3500 40  0000 C CNN
+F 0 "R2" V 1430 3500 40  0000 C CNN
 F 1 "R" V 1357 3501 40  0000 C CNN
 F 2 "~" V 1280 3500 30  0000 C CNN
@@
 $EndComp
 $Comp
-L LED D2
+L LED D1
 U 1 1 54CE50E1
 P 950 1450
-F 0 "D2" H 950 1550 50  0000 C CNN
+F 0 "D1" H 950 1550 50  0000 C CNN
 F 1 "PWRSTAT" H 950 1350 50  0000 C CNN
 F 2 "~" H 950 1450 60  0000 C CNN
