File: hardware/APRSDongle.kicad_pcb (KiCad board)
At the start: 2 copper layers, 26 parts, among them IC1 DRA818, J1 SMA, P1 VIN, P2 GPS, P3 PC_CON, P4 CONN_8, P5 SWD, U1 AP7363, U2 KL05

Commit message: added a fill to top and bottom. Ground
Routing:
- net GND: track 150.8 -> 153.1 mm, vias 3 -> 4
- added copper zone on F.Cu, net GND
- removed copper zone on F.Cu, net (none)
Changed lines of the file:
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@@
     (thickness 1.6)
     (drawings 0)
-    (tracks 254)
+    (tracks 259)
     (zones 0)
     (modules 26)
@@
     )
   )
-  (segment (start 374.714 244) (end 373.2 244) (width 0.7) (layer B.Cu) (net 1) (status 400000))
-  (segment (start 367.41 245.6) (end 364.81 243) (width 0.7) (layer B.Cu) (net 1) (status 800000))
+  (segment (start 374.714 244) (end 373.2 244) (width 0.7) (layer B.Cu) (net 1))
+  (segment (start 367.41 245.6) (end 364.81 243) (width 0.7) (layer B.Cu) (net 1))
   (segment (start 371.6 245.6) (end 367.41 245.6) (width 0.7) (layer B.Cu) (net 1))
   (segment (start 373.2 244) (end 371.6 245.6) (width 0.7) (layer B.Cu) (net 1))
-  (segment (start 374.714 244) (end 375.8 244) (width 0.7) (layer B.Cu) (net 1) (status 400000))
-  (segment (start 375.3525 241.5525) (end 375 241.5525) (width 0.7) (layer F.Cu) (net 1) (status C00000))
-  (segment (start 376.8 243) (end 375.3525 241.5525) (width 0.7) (layer F.Cu) (net 1) (status 800000))
+  (segment (start 374.714 244) (end 375.8 244) (width 0.7) (layer B.Cu) (net 1))
+  (segment (start 375.3525 241.5525) (end 375 241.5525) (width 0.7) (layer F.Cu) (net 1))
+  (segment (start 376.8 243) (end 375.3525 241.5525) (width 0.7) (layer F.Cu) (net 1))
   (via (at 376.8 243) (size 0.889) (layers F.Cu B.Cu) (net 1))
   (segment (start 375.8 244) (end 376.8 243) (width 0.7) (layer B.Cu) (net 1))
@@
   (segment (start 339.97308 223.02692) (end 341.174 223.02692) (width 0.254) (layer F.Cu) (net 20))
   (segment (start 339.73 223.27) (end 339.97308 223.02692) (width 0.254) (layer F.Cu) (net 20))
-  (segment (start 347.9525 231) (end 347.9525 233.7525) (width 0.7) (layer F.Cu) (net 21) (status 400000))
+  (via (at 377 237.65) (size 0.889) (layers F.Cu B.Cu) (net 21))
+  (segment (start 380 228) (end 379 229) (width 0.7) (layer F.Cu) (net 21))
+  (segment (start 379 229) (end 379 233) (width 0.7) (layer F.Cu) (net 21))
+  (via (at 379 233) (size 0.889) (layers F.Cu B.Cu) (net 21))
+  (segment (start 379 233) (end 377 235) (width 0.7) (layer B.Cu) (net 21))
+  (segment (start 377 235) (end 377 237.65) (width 0.7) (layer B.Cu) (net 21))
+  (segment (start 382.8 228) (end 380 228) (width 0.7) (layer F.Cu) (net 21))
+  (segment (start 377 237.65) (end 377 239.6475) (width 0.7) (layer F.Cu) (net 21))
+  (segment (start 377 239.6475) (end 377 239.8) (width 0.7) (layer F.Cu) (net 21))
+  (segment (start 377 239.8) (end 377 239.6475) (width 0.7) (layer F.Cu) (net 21))
+  (segment (start 347.9525 231) (end 347.9525 233.7525) (width 0.7) (layer F.Cu) (net 21))
   (via (at 349.6 243) (size 0.889) (layers F.Cu B.Cu) (net 21))
   (segment (start 349.6 235.4) (end 349.6 243) (width 0.7) (layer B.Cu) (net 21))
@@
   (segment (start 349.6 242.9525) (end 349.6 243) (width 0.7) (layer F.Cu) (net 21))
   (segment (start 349.6 243) (end 349.6 242.9525) (width 0.7) (layer F.Cu) (net 21))
-  (segment (start 342.27 238.5) (end 342.27 241.04) (width 0.7) (layer F.Cu) (net 21) (status C00000))
-  (segment (start 375 239.6475) (end 374.6225 239.6475) (width 0.7) (layer F.Cu) (net 21) (status C00000))
-  (segment (start 374.6225 239.6475) (end 371.27 243) (width 0.7) (layer F.Cu) (net 21) (status C00000))
-  (segment (start 378.6 239.6475) (end 381.84746 239.6475) (width 0.7) (layer F.Cu) (net 21) (status 400000))
-  (segment (start 381.84746 239.6475) (end 382.69998 240.50002) (width 0.7) (layer F.Cu) (net 21) (status 800000))
-  (segment (start 378.6 239.6475) (end 375 239.6475) (width 0.7) (layer F.Cu) (net 21) (status C00000))
+  (segment (start 342.27 238.5) (end 342.27 241.04) (width 0.7) (layer F.Cu) (net 21))
+  (segment (start 375 239.6475) (end 374.6225 239.6475) (width 0.7) (layer F.Cu) (net 21))
+  (segment (start 374.6225 239.6475) (end 371.27 243) (width 0.7) (layer F.Cu) (net 21))
+  (segment (start 378.6 239.6475) (end 381.84746 239.6475) (width 0.7) (layer F.Cu) (net 21))
+  (segment (start 381.84746 239.6475) (end 382.69998 240.50002) (width 0.7) (layer F.Cu) (net 21))
+  (segment (start 378.6 239.6475) (end 377 239.6475) (width 0.7) (layer F.Cu) (net 21))
+  (segment (start 377 239.6475) (end 375 239.6475) (width 0.7) (layer F.Cu) (net 21))
   (segment (start 389.47 209.8) (end 389 209.8) (width 0.4) (layer F.Cu) (net 21))
   (segment (start 384.1525 208.6) (end 382.7525 210) (width 0.4) (layer F.Cu) (net 21))
@@
   (segment (start 387.2 226.8) (end 386 228) (width 0.7) (layer F.Cu) (net 21))
   (segment (start 386 228) (end 382.8 228) (width 0.7) (layer F.Cu) (net 21))
-  (segment (start 382.8 228) (end 380 228) (width 0.7) (layer F.Cu) (net 21))
-  (segment (start 377 235) (end 377 237.65) (width 0.7) (layer B.Cu) (net 21))
-  (segment (start 379 233) (end 377 235) (width 0.7) (layer B.Cu) (net 21))
-  (via (at 379 233) (size 0.889) (layers F.Cu B.Cu) (net 21))
-  (segment (start 379 229) (end 379 233) (width 0.7) (layer F.Cu) (net 21))
-  (segment (start 380 228) (end 379 229) (width 0.7) (layer F.Cu) (net 21))
   (segment (start 389.5 215.85) (end 387.95 215.85) (width 0.7) (layer F.Cu) (net 22))
   (segment (start 379.27 212) (end 377.27 210) (width 0.7) (layer F.Cu) (net 22))
@@
   (segment (start 386.93 212.62) (end 385.4 214.15) (width 0.254) (layer F.Cu) (net 30))
   (segment (start 368.73 238) (end 368.73 243) (width 0.7) (layer F.Cu) (net 31))
-  (segment (start 371.27 238) (end 371.27 239.87) (width 0.7) (layer B.Cu) (net 32) (status 400000))
-  (segment (start 376.886 241.6) (end 379.286 244) (width 0.7) (layer B.Cu) (net 32) (status 800000))
+  (segment (start 371.27 238) (end 371.27 239.87) (width 0.7) (layer B.Cu) (net 32))
+  (segment (start 376.886 241.6) (end 379.286 244) (width 0.7) (layer B.Cu) (net 32))
   (segment (start 373 241.6) (end 376.886 241.6) (width 0.7) (layer B.Cu) (net 32))
   (segment (start 371.27 239.87) (end 373 241.6) (width 0.7) (layer B.Cu) (net 32))
-  (segment (start 378.6 241.5525) (end 379.9525 241.5525) (width 0.7) (layer F.Cu) (net 32) (status 400000))
-  (segment (start 380 244) (end 379.286 244) (width 0.7) (layer B.Cu) (net 32) (status C00000))
-  (segment (start 380.8 243.2) (end 380 244) (width 0.7) (layer B.Cu) (net 32) (status 800000))
+  (segment (start 378.6 241.5525) (end 379.9525 241.5525) (width 0.7) (layer F.Cu) (net 32))
+  (segment (start 380 244) (end 379.286 244) (width 0.7) (layer B.Cu) (net 32))
+  (segment (start 380.8 243.2) (end 380 244) (width 0.7) (layer B.Cu) (net 32))
   (via (at 380.8 243.2) (size 0.889) (layers F.Cu B.Cu) (net 32))
   (segment (start 380.8 242.4) (end 380.8 243.2) (width 0.7) (layer F.Cu) (net 32))
@@
     )
   )
-  (zone (net 0) (net_name "") (layer F.Cu) (hatch edge 0.508)
-    (connect_pads yes (clearance 0.17))
+  (zone (net 21) (net_name GND) (layer F.Cu) (hatch edge 0.508)
+    (connect_pads (clearance 0.17))
     (min_thickness 0.254)
     (fill (arc_segments 16) (thermal_gap 0.508) (thermal_bridge_width 0.508))
     (polygon
       (pts
-        (xy 379.2 218.8) (xy 379.2 227) (xy 385.8 226.8) (xy 387.2 225.8) (xy 387.4 218.8)
+        (xy 392.4 246.4) (xy 392.4 208.2) (xy 337.6 208.2) (xy 337.6 246.4)
       )
     )
-  )
-  (zone (net 0) (net_name "") (layer F.Cu) (hatch edge 0.508)
-    (connect_pads yes (clearance 0.17))
-    (min_thickness 0.254)
-    (fill (arc_segments 16) (thermal_gap 0.508) (thermal_bridge_width 0.508))
-    (polygon
-      (pts
-        (xy 356.8 219.8) (xy 355.6 221.8) (xy 353 221) (xy 353.2 214.4) (xy 354.4 212.6)
-        (xy 356.6 212.6)
-      )
-    )
-  )
-  (zone (net 0) (net_name "") (layer F.Cu) (hatch edge 0.508)
-    (connect_pads yes (clearance 0.17))
-    (min_thickness 0.254)
-    (fill (arc_segments 16) (thermal_gap 0.508) (thermal_bridge_width 0.508))
-    (polygon
-      (pts
-        (xy 353 228.2) (xy 353.2 232.6) (xy 356.2 234.2) (xy 357.2 228.6) (xy 356.6 226)
-        (xy 356.4 225.4) (xy 353.8 225.4)
-      )
-    )

Commit message: had to fix the netlise.... just dont reanotate. A few more changes, not much
Connections:
- DRAC1 pad 1: +3.3V -> N-0000043
- DRAPOW1 pad 2: N-000001 (its old number) -> N-0000043
- IC1 pad 8: N-000001 (its old number) -> N-0000043
Routing:
- net N-0000043: track 0.00 -> 19.5 mm
- net N-000001 (its old number): track 17.2 -> 0.00 mm
- net +3.3V: track 121.1 -> 113.8 mm

Commit message: this commit is the real one. the last one was a lie
Parts:
- moved DRAC1 12.3 mm to (391.2, 218.0), turned to 270 degrees
- moved IC1 0.80 mm to (353.2, 232.2)
- renumbered P5 to ProgHead
Routing:
- net GND: track 153.1 -> 147.0 mm, vias 4 -> 29
- net N-0000043: track 19.5 -> 20.3 mm
- net /ADC0_6: track 18.7 -> 19.4 mm
Other:
- board outline added: 54.8 x 38.6 mm
- board text added: "AB1TJ APRSDongle"
