File: hardware/hardwareRev1.sch (KiCad schematic (older format))
At the start: 59 parts, among them J1 MicroSD, J2 SMA, K1 PWMOut, K2 ADC1, P1 UART, P10 ID, P2 I2C, P3 ADC2, P4 CONN_7, P5 CONN_5X2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

Commit message: Really really large commit because I like to live dangerously...
Parts:
- C1, C10, C11, C12, C13, C14, C2, C3, C4, C5, C6, C8, C9: symbol C -> C-RESCUE-hardwareRev1
- D1, D2, D3, D4: symbol LED -> LED-RESCUE-hardwareRev1
- R1, R10, R11, R12, R13, R14, R2, R3, R4, R5, R6, R7, R8, R9: symbol R -> R-RESCUE-hardwareRev1
