File: hardwareRev1/hardwareRev1.sch (KiCad schematic (older format))
At the start: 10 parts

Commit message: did more things.
Parts:
- added A?: GPSAnt, gpsAnt, symbol GPSAnt
- added C?: C, symbol C
- added JMP? (x2): SJMPOpen, symbol SJMPOpen
- added TP? (x3): TEST-POINT2, SparkFun-PAD.02X.02, symbol TEST-POINT2
- added TP?: USBIN, SparkFun-PAD.02X.02, symbol TEST-POINT2
- added TP?: 3v3Out, SparkFun-PAD.02X.02, symbol TEST-POINT2
- added U?: MICRO-B_USB, symbol MICRO-B_USB
Connections:
- net labels added: USBDM, USBDP, USBV1, USBV2, gpsPulse, gpsRx, gpsTX, internalI2CSCL, internalI2CSDA
- wire segments 83 -> 112
- no-connect marks 0 -> 5
Other:
- moved on the sheet: RF?

Commit message: getting pretty far with the next revision.
Parts:
- removed P?: PWRIN, symbol CONN_9X2
- added C10, C2, C3, C4, C5: C, Capacitors_SMD:C_0603, symbol C
- added JMP1: SJMPOpen, symbol SJMPOpen
- added P1: CONN_5X2, symbol CONN_5X2
- added P?: CONN_11X2, symbol CONN_11X2
- added Q1: MOSFET_P, symbol MOSFET_P
- added R1, R2, R3: R, symbol R
- added X1: CRYSTAL_ABM3C, symbol CRYSTAL_ABM3C
- C1, C6, C7, C8, C9: renamed from C?; footprint (none) -> Capacitors_SMD:C_0603
- TP2: renamed from TP?; value TEST-POINT2 -> GPSDM
- TP3: renamed from TP?; value TEST-POINT2 -> GPSDP
- gave numbers to parts that had none: 12
Connections:
- net labels added: GPSPulse, GPSRX, GPSTX, GPSTx, SDPower, SWD_CLK, SWD_DIO, SWD_RST, SWD_Reset, externalI2C1SCL, externalI2C1SDA, externalSPI1MISO, externalSPI1MOSI, externalUART2RX, externalUART2TX, internalI2C0SCL, internalI2C0SDA, internalSPI0Clk, internalSPI0MISO, internalSPI0MOSI, internalSPI0SCK
- net labels removed: gpsPulse, gpsRx, gpsTX, internalSPIClk, internalSPIMISO, internalSPIMOSI
- wire segments 112 -> 218
Other:
- moved on the sheet: A1, C1, U1

Commit message: board is almost done. Commiting before I destroy all my work...
Parts:
- removed Q1: MOSFET_P, symbol MOSFET_P
- removed TP1: 3v3Out, SparkFun-PAD.02X.02, symbol TEST-POINT2
- removed TP2: GPSDM, SparkFun-PAD.02X.02, symbol TEST-POINT2
- removed TP3: GPSDP, SparkFun-PAD.02X.02, symbol TEST-POINT2
- removed TP4: USBIN, SparkFun-PAD.02X.02, symbol TEST-POINT2
- removed TP5: TEST-POINT2, SparkFun-PAD.02X.02, symbol TEST-POINT2
- added C11, C12, C13: C, Capacitors_SMD:C_0603, symbol C
- added D1, D2, D3, D4: LED, LEDs:LED-0805, symbol LED
- added D5: DIODE, Diodes_ThroughHole:Diode_DO-41_SOD81_Vertical_AnodeUp, symbol DIODE
- added K1: PWMOut, Footprints:CONN_1x3, symbol CONN_3
- added K2: ADC1, Footprints:CONN_1x3, symbol CONN_3
- added P1: UART, Footprints:CONN_1x4, symbol CONN_4
- added P10: ID, Measurement_Points:Measurement_Point_Round-SMD-Pad_Small, symbol CONN_1
- added P2: I2C, Footprints:CONN_1x4, symbol CONN_4
- added P3: ADC2, Footprints:CONN_1x5, symbol CONN_5
- added P4: CONN_7, Footprints:CONN_1x7, symbol CONN_7
- added P7: GPSDM, Measurement_Points:Measurement_Point_Round-SMD-Pad_Small, symbol CONN_1
- added P8: GPSDP, Measurement_Points:Measurement_Point_Round-SMD-Pad_Small, symbol CONN_1
- added P9: USBPW, Measurement_Points:Measurement_Point_Round-SMD-Pad_Small, symbol CONN_1
- added Q1: MOS_P_NUM, SMD_Packages:SOT-323, symbol MOS_P_NUM
- added R1, R11, R12, R13, R2, R3, R4, R5, R6, R8: R, Resistors_SMD:R_0603, symbol R
- added S1, S2: TAC_SWITCHSMD, SparkFun:SparkFun-TACTILE_SWITCH_SMD, symbol TAC_SWITCHSMD
- added U2: 24C16, Housings_SOIC:SOIC-8_3.9x4.9mm_Pitch1.27mm, symbol 24C16
- A1: footprint gpsAnt -> hardwareRev1:GPSAnt
- J1: footprint (none) -> Footprints:MICRO_SD_HINGE_AMP
- J2: footprint SMA -> hardwareRev1:SMA
- JMP1, JMP2, JMP3: footprint (none) -> SparkFun:SparkFun-SJ_2S-NO
- P5: renamed from P1; footprint (none) -> hardwareRev1:CortexDebug
- P6: renamed from P?; footprint (none) -> hardwareRev1:1.27mmPitchHeader11X2
- R10: renamed from R3; footprint (none) -> Resistors_SMD:R_0603
- R7: renamed from R1; footprint (none) -> Resistors_SMD:R_0603
- R9: renamed from R2; footprint (none) -> Resistors_SMD:R_0603
- RF1: footprint (none) -> hardwareRev1:NEO-7
- RF2: footprint (none) -> dra818:DRA818
- U1: footprint MODULE -> w_smd_lqfp:lqfp64
- U3: renamed from U2; footprint (none) -> USB:USB micro B female
- X1: footprint (none) -> open-project:CRYSTAL_ABM3C
Connections:
- net labels added: LED1, LED2, LED3, LED4, SW0, SW1, externalADC1, externalADC2, externalADC3, externalADC4, externalPWMOut, externalSPI1CS1, externalSPI1PCS0, externalSPI1SCK, internalI2C1SCL, internalI2C1SDA
- net labels removed: SWD_RST, internalI2CSCL, internalI2CSDA, internalSPI0SCK
- wire segments 218 -> 318
- no-connect marks 5 -> 28
Other:
- moved on the sheet: A1

Commit message: went further.
Connections:
- net labels removed: PWRSDA, PwrCLK, PwrSDA
- wire segments 318 -> 322

Commit message: better routed it.
Parts:
- removed P9: USBPW, Measurement_Points:Measurement_Point_Round-SMD-Pad_Small, symbol CONN_1
Changed lines of the file:
@@
 EESchema Schematic File Version 2
+LIBS:hardwareRev1-rescue
 LIBS:power
 LIBS:device
@@
 LIBS:contrib
 LIBS:valves
+LIBS:MKL26Z128VLH4
+LIBS:USB
+LIBS:sma
+LIBS:DataStorage
+LIBS:dra818Real
+LIBS:SparkFun
+LIBS:neo7
+LIBS:gpsant
+LIBS:open-project
+LIBS:smtJmpOpen
 LIBS:conn_11x2
-LIBS:tps63020
-LIBS:ncp508
-LIBS:smtJmpOpen
-LIBS:SparkFun
-LIBS:attiny24a-m
-LIBS:power-cache
+LIBS:MOS_P_NUM
+LIBS:hardwareRev1-cache
 EELAYER 25 0
 EELAYER END
@@
 SW0
 $Comp
-L CONN_1 P9
-U 1 1 554D49E1
-P 7250 5700
-F 0 "P9" H 7330 5700 40  0000 L CNN
-F 1 "USBPW" H 7250 5755 30  0001 C CNN
-F 2 "Measurement_Points:Measurement_Point_Round-SMD-Pad_Small" H 7250 5700 60  0001 C CNN
-F 3 "" H 7250 5700 60  0000 C CNN
-	1    7250 5700
-	0    1    1    0
-$EndComp
-$Comp
 L CONN_1 P10

Commit message: board is done. Onto the radio module
Parts:
- added C14: C, Capacitors_ThroughHole:C_Rect_L13_W6_H12_P10, symbol C
- added R14: R, Resistors_SMD:R_0603, symbol R
Connections:
- net labels removed: internalI2C1SCL, internalI2C1SDA
- wire segments 322 -> 327
Changed lines of the file:
@@
 L +3.3V #PWR014
 U 1 1 5546BB95
-P 8400 1100
-F 0 "#PWR014" H 8400 1060 30  0001 C CNN
-F 1 "+3.3V" H 8400 1210 30  0000 C CNN
-F 2 "" H 8400 1100 60  0000 C CNN
-F 3 "" H 8400 1100 60  0000 C CNN
-	1    8400 1100
+P 8600 1450
+F 0 "#PWR014" H 8600 1410 30  0001 C CNN
+F 1 "+3.3V" H 8600 1560 30  0000 C CNN
+F 2 "" H 8600 1450 60  0000 C CNN
+F 3 "" H 8600 1450 60  0000 C CNN
+	1    8600 1450
 	1    0    0    -1
 $EndComp
@@
 NoConn ~ 6450 3550
 Text Label 5900 750  0    60   ~ 0
-internalI2C1SDA
+internalI2C0SDA
 Text Label 5900 850  0    60   ~ 0
-internalI2C1SCL
+internalI2C0SCL
 Text Label 5900 950  0    60   ~ 0
 GPSTX
@@
 Connection ~ 9000 2350
 Wire Wire Line
-	8250 1250 8400 1250
-Wire Wire Line
-	8400 1100 8400 1400
-Wire Wire Line
 	8400 1400 8250 1400
-Connection ~ 8400 1250
 Wire Wire Line
 	8250 1700 8400 1700
@@
 	8350 5250 8350 5300
 Connection ~ 8350 5300
+$Comp
+L C C14
+U 1 1 554FE992
+P 9450 1250
+F 0 "C14" H 9450 1350 40  0000 L CNN
+F 1 "C" H 9456 1165 40  0000 L CNN
+F 2 "Capacitors_ThroughHole:C_Rect_L13_W6_H12_P10" H 9488 1100 30  0001 C CNN
+F 3 "" H 9450 1250 60  0000 C CNN
+	1    9450 1250
+	1    0    0    -1
+$EndComp
+$Comp
+L R R14
+U 1 1 554FECB3
+P 9050 1500
+F 0 "R14" V 9130 1500 40  0000 C CNN
+F 1 "R" V 9057 1501 40  0000 C CNN
+F 2 "Resistors_SMD:R_0603" V 8980 1500 30  0001 C CNN
+F 3 "" H 9050 1500 30  0000 C CNN
+	1    9050 1500
+	0    1    1    0
+$EndComp
+Wire Wire Line
+	8400 1400 8400 1500
+Wire Wire Line
+	8400 1500 8800 1500
+Wire Wire Line
+	8600 1500 8600 1450
+Connection ~ 8600 1500
+Wire Wire Line
+	9300 1500 9450 1500
+Wire Wire Line
+	9450 1500 9450 1450
+Wire Wire Line
+	9450 1050 8250 1050
+Wire Wire Line
+	8250 1050 8250 1250
 $EndSCHEMATC
