File: hardwareRev1/Radio/radio.sch (KiCad schematic (older format))
At the start: 0 parts

Commit message: almost done with radio schematic
Parts:
- added C?: 2.2pf, symbol C
- added C?: 22pf, symbol C
- added C?: 33pf, symbol C
- added C?: 47pf, symbol C
- added C?: 15pf, symbol C
- added C?: 4.7pf, symbol C
- added C?: 1.8pf, symbol C
- added C? (x4): 10pf, symbol C
- added C? (x2): 12pf, symbol C
- added C? (x8): C, symbol C
- added L?: 150nh, symbol INDUCTOR
- added L? (x3): 120nH, symbol INDUCTOR
- added L?: 39nH, symbol INDUCTOR
- added L?: 47nH, symbol INDUCTOR
- added L? (x2): 150nH, symbol INDUCTOR
- added L? (x2): 68nH, symbol INDUCTOR
- added L? (x2): INDUCTOR, symbol INDUCTOR
- added R?: R, symbol R
- added U?: AX503, MODULE, symbol AX503
- added U?: RF5110G, MODULE, symbol RF5110G
- added U?: PE42424, MODULE, symbol PE42424
- added X?: TCXO, symbol TCXO
Connections:
- net labels added: +3.3V, AF_IN, AF_OUT, CLK, GND, IRQOUT, MISO, MOSI, SEL, TXRX, UART_RX, UART_TX
- wire segments 0 -> 107
- no-connect marks 0 -> 1
