File: hardwareRev1/Radio/MCU.sch (KiCad schematic (older format))
At the start: 34 parts

Commit message: Made the board 4 layer.
Added a MCU to theback...
Parts:
- removed P?: I2C, Footprints:CONN_1x4, symbol CONN_4
- removed S?: TAC_SWITCHSMD, SparkFun:SparkFun-TACTILE_SWITCH_SMD, symbol TAC_SWITCHSMD
- removed U?: 24C16, Housings_SOIC:SOIC-8_3.9x4.9mm_Pitch1.27mm, symbol 24C16
- C38, C39, C40, C41, C42: renamed from C?; footprint Capacitors_SMD:C_0603 -> Capacitors_SMD:C_0402
- C43: renamed from C?; footprint (none) -> Capacitors_SMD:C_0402
- C44: renamed from C?; footprint Capacitors_ThroughHole:C_Rect_L13_W6_H12_P10 -> FC0H224ZFTBR24:FC0H224ZFTBR24
- D1, D2: renamed from D?; footprint LEDs:LED-0805 -> LEDs:LED-0603
- D3: renamed from D?; footprint (none) -> Diodes_SMD:SOD-323
- J2: renamed from J?; footprint SMA -> hardwareRev1:EdgeSMA
- JMP1, JMP3, JMP4: renamed from JMP?; footprint SparkFun:SparkFun-SJ_2S-NO -> hardwareRev1:SMDJMP-OPEN
- JMP2: renamed from JMP?; footprint (none) -> hardwareRev1:SMDJMP-CLOSED
- L16: renamed from L?; footprint (none) -> Resistors_SMD:R_0402
- P3: renamed from P?; value CONN_7 -> CONN_8; footprint Footprints:CONN_1x7 -> Connectors_Molex:Connector_Molex_PicoBlade_53398-0871; symbol CONN_7 -> CONN_8
- R2, R3, R4, R5, R6, R8: renamed from R?; footprint Resistors_SMD:R_0603 -> Resistors_SMD:R_0402
- R7: renamed from R?; footprint (none) -> Resistors_SMD:R_0402
- RF2: renamed from RF?; footprint (none) -> hardwareRev1:NEO-7
- gave numbers to parts that had none: 6
Connections:
- net labels added: externalSPI1CS2
- wire segments 184 -> 175
- no-connect marks 13 -> 11
