File: hardwareRev1/Radio/PA.sch (KiCad schematic (older format))
At the start: 34 parts, among them U3 RF5110G

Commit message: Made the board 4 layer.
Added a MCU to theback...
Parts:
- C33: renamed from C37; footprint (none) -> Capacitors_SMD:C_0402
- renumbered C13 to C14, C14 to C15, C15 to C16, C16 to C17, C17 to C18, C18 to C19, C19 to C20, C20 to C21, C21 to C22, C22 to C23, C23 to C24, C24 to C25, C25 to C26, C26 to C27, C27 to C28, C28 to C29, C29 to C30, C30 to C31, C31 to C32, C32 to C34, C33 to C35, C34 to C36, C35 to C37, R2 to R1
Changed lines of the file:
@@
 $Descr A4 11693 8268
 encoding utf-8
-Sheet 2 3
+Sheet 2 2
 Title ""
 Date ""
@@
 $EndComp
 $Comp
-L C C13
+L C C14
 U 1 1 55503CBD
 P 1650 6200
-F 0 "C13" H 1650 6300 40  0000 L CNN
+F 0 "C14" H 1650 6300 40  0000 L CNN
 F 1 "2.2pf" H 1656 6115 40  0000 L CNN
 F 2 "Capacitors_SMD:C_0402" H 1688 6050 30  0001 C CNN
@@
 $EndComp
 $Comp
-L C C14
+L C C15
 U 1 1 55503CE0
 P 2250 5950
-F 0 "C14" H 2250 6050 40  0000 L CNN
+F 0 "C15" H 2250 6050 40  0000 L CNN
 F 1 "22pf" H 2256 5865 40  0000 L CNN
 F 2 "Capacitors_SMD:C_0402" H 2288 5800 30  0001 C CNN
@@
 $EndComp
 $Comp
-L C C15
+L C C16
 U 1 1 55503D9F
 P 3350 6200
-F 0 "C15" H 3350 6300 40  0000 L CNN
+F 0 "C16" H 3350 6300 40  0000 L CNN
 F 1 "33pf" H 3356 6115 40  0000 L CNN
 F 2 "Capacitors_SMD:C_0402" H 3388 6050 30  0001 C CNN
@@
 $EndComp
 $Comp
-L C C17
+L C C18
 U 1 1 55503DFA
 P 4150 6200
-F 0 "C17" H 4150 6300 40  0000 L CNN
+F 0 "C18" H 4150 6300 40  0000 L CNN
 F 1 "47pf" H 4156 6115 40  0000 L CNN
 F 2 "Capacitors_SMD:C_0402" H 4188 6050 30  0001 C CNN
@@
 $EndComp
 $Comp
-L C C22
+L C C23
 U 1 1 55503E1E
 P 4950 6200
-F 0 "C22" H 4950 6300 40  0000 L CNN
+F 0 "C23" H 4950 6300 40  0000 L CNN
 F 1 "15pf" H 4956 6115 40  0000 L CNN
 F 2 "Capacitors_SMD:C_0402" H 4988 6050 30  0001 C CNN
@@
 $EndComp
 $Comp
-L C C16
+L C C17
 U 1 1 55503E3F
 P 3750 5600
-F 0 "C16" H 3750 5700 40  0000 L CNN
+F 0 "C17" H 3750 5700 40  0000 L CNN
 F 1 "4.7pf" H 3756 5515 40  0000 L CNN
 F 2 "Capacitors_SMD:C_0402" H 3788 5450 30  0001 C CNN
@@
 $EndComp
 $Comp
-L C C20
+L C C21
 U 1 1 55503E69
 P 4500 5600
-F 0 "C20" H 4500 5700 40  0000 L CNN
+F 0 "C21" H 4500 5700 40  0000 L CNN
 F 1 "1.8pf" H 4506 5515 40  0000 L CNN
 F 2 "Capacitors_SMD:C_0402" H 4538 5450 30  0001 C CNN
@@
 $EndComp
 $Comp
-L GND #PWR25
+L GND #PWR055
 U 1 1 55503EBE
 P 1650 6900
-F 0 "#PWR25" H 1650 6900 30  0001 C CNN
+F 0 "#PWR055" H 1650 6900 30  0001 C CNN
 F 1 "GND" H 1650 6830 30  0001 C CNN
 F 2 "" H 1650 6900 60  0000 C CNN
@@
 $EndComp
 $Comp
-L GND #PWR26
+L GND #PWR056
 U 1 1 55503EDE
 P 3350 6750
-F 0 "#PWR26" H 3350 6750 30  0001 C CNN
+F 0 "#PWR056" H 3350 6750 30  0001 C CNN
 F 1 "GND" H 3350 6680 30  0001 C CNN
 F 2 "" H 3350 6750 60  0000 C CNN
@@
 $EndComp
 $Comp
-L GND #PWR28
+L GND #PWR057
 U 1 1 55503EFE
 P 4150 6700
-F 0 "#PWR28" H 4150 6700 30  0001 C CNN
+F 0 "#PWR057" H 4150 6700 30  0001 C CNN
 F 1 "GND" H 4150 6630 30  0001 C CNN
 F 2 "" H 4150 6700 60  0000 C CNN
@@
 $EndComp
 $Comp
-L GND #PWR30
+L GND #PWR058
 U 1 1 55503F1E
 P 4950 6750
-F 0 "#PWR30" H 4950 6750 30  0001 C CNN
+F 0 "#PWR058" H 4950 6750 30  0001 C CNN
 F 1 "GND" H 4950 6680 30  0001 C CNN
 F 2 "" H 4950 6750 60  0000 C CNN
@@
 $EndComp
 $Comp
-L R R2
+L R R1
 U 1 1 55508666
 P 5450 6200
-F 0 "R2" V 5530 6200 40  0000 C CNN
+F 0 "R1" V 5530 6200 40  0000 C CNN
 F 1 "180" V 5457 6201 40  0000 C CNN
 F 2 "Resistors_SMD:R_0402" V 5380 6200 30  0001 C CNN
@@
 $EndComp
 $Comp
-L C C25
+L C C26
 U 1 1 555086C4
 P 5850 5800
-F 0 "C25" H 5850 5900 40  0000 L CNN
+F 0 "C26" H 5850 5900 40  0000 L CNN
 F 1 "100pf" H 5856 5715 40  0000 L CNN
 F 2 "Capacitors_SMD:C_0402" H 5888 5650 30  0001 C CNN
@@
 $EndComp
 $Comp
-L C C21
+L C C22
 U 1 1 55508E11
 P 4950 3150
-F 0 "C21" H 4950 3250 40  0000 L CNN
+F 0 "C22" H 4950 3250 40  0000 L CNN
 F 1 "10nf" H 4956 3065 40  0000 L CNN
 F 2 "Capacitors_SMD:C_0402" H 4988 3000 30  0001 C CNN
@@
 $EndComp
 $Comp
-L C C23
+L C C24
 U 1 1 55508E7A
 P 5150 3150
-F 0 "C23" H 5150 3250 40  0000 L CNN
+F 0 "C24" H 5150 3250 40  0000 L CNN
 F 1 "1nf" H 5156 3065 40  0000 L CNN
 F 2 "Capacitors_SMD:C_0402" H 5188 3000 30  0001 C CNN
@@
 $EndComp
 $Comp
-L C C24
+L C C25
 U 1 1 55508EB6
 P 5350 3150
-F 0 "C24" H 5350 3250 40  0000 L CNN
+F 0 "C25" H 5350 3250 40  0000 L CNN
 F 1 "27pf" H 5356 3065 40  0000 L CNN
 F 2 "Capacitors_SMD:C_0402" H 5388 3000 30  0001 C CNN
@@
 $EndComp
 $Comp
-L GND #PWR29
+L GND #PWR059
 U 1 1 55508EF7
 P 4950 3550
-F 0 "#PWR29" H 4950 3550 30  0001 C CNN
+F 0 "#PWR059" H 4950 3550 30  0001 C CNN
 F 1 "GND" H 4950 3480 30  0001 C CNN
 F 2 "" H 4950 3550 60  0000 C CNN
@@
 $EndComp
 $Comp
-L C C26
+L C C27
 U 1 1 5550A0C6
 P 6100 2600
-F 0 "C26" H 6100 2700 40  0000 L CNN
+F 0 "C27" H 6100 2700 40  0000 L CNN
 F 1 "27pf" H 6106 2515 40  0000 L CNN
 F 2 "Capacitors_SMD:C_0402" H 6138 2450 30  0001 C CNN
@@
 $EndComp
 $Comp
-L C C28
+L C C29
 U 1 1 5550A155
 P 6900 3100
-F 0 "C28" H 6900 3200 40  0000 L CNN
+F 0 "C29" H 6900 3200 40  0000 L CNN
 F 1 "1nf" H 6906 3015 40  0000 L CNN
 F 2 "Capacitors_SMD:C_0402" H 6938 2950 30  0001 C CNN
@@
 $EndComp
 $Comp
-L C C29
+L C C30
 U 1 1 5550A1A9
 P 7200 3100
-F 0 "C29" H 7200 3200 40  0000 L CNN
+F 0 "C30" H 7200 3200 40  0000 L CNN
 F 1 "10nf" H 7206 3015 40  0000 L CNN
 F 2 "Capacitors_SMD:C_0402" H 7238 2950 30  0001 C CNN
@@
 $EndComp
 $Comp
-L C C31
+L C C32
 U 1 1 5550A1EA
 P 7450 3100
-F 0 "C31" H 7450 3200 40  0000 L CNN
+F 0 "C32" H 7450 3200 40  0000 L CNN
 F 1 "3.3uf" H 7456 3015 40  0000 L CNN
 F 2 "Capacitors_SMD:C_1206" H 7488 2950 30  0001 C CNN
@@
 $EndComp
 $Comp
-L GND #PWR35
+L GND #PWR060
 U 1 1 5550A22C
 P 7250 3400
-F 0 "#PWR35" H 7250 3400 30  0001 C CNN
+F 0 "#PWR060" H 7250 3400 30  0001 C CNN
 F 1 "GND" H 7250 3330 30  0001 C CNN
 F 2 "" H 7250 3400 60  0000 C CNN
@@
 $EndComp
 $Comp
-L GND #PWR31
+L GND #PWR061
 U 1 1 5550A374
 P 6250 2450
-F 0 "#PWR31" H 6250 2450 30  0001 C CNN
+F 0 "#PWR061" H 6250 2450 30  0001 C CNN
 F 1 "GND" H 6250 2380 30  0001 C CNN
 F 2 "" H 6250 2450 60  0000 C CNN
@@
 $EndComp
 $Comp
-L C C27
+L C C28
 U 1 1 5550B492
 P 6550 3400
-F 0 "C27" H 6550 3500 40  0000 L CNN
+F 0 "C28" H 6550 3500 40  0000 L CNN
 F 1 "47pf" H 6556 3315 40  0000 L CNN
 F 2 "Capacitors_SMD:C_0402" H 6588 3250 30  0001 C CNN
@@
 $EndComp
 $Comp
-L GND #PWR34
+L GND #PWR062
 U 1 1 5550B4DF
 P 6550 3750
-F 0 "#PWR34" H 6550 3750 30  0001 C CNN
+F 0 "#PWR062" H 6550 3750 30  0001 C CNN
 F 1 "GND" H 6550 3680 30  0001 C CNN
 F 2 "" H 6550 3750 60  0000 C CNN
@@
 $EndComp
 $Comp
-L +3.3V #PWR33
+L +3.3V #PWR063
 U 1 1 5550B51F
 P 6300 3100
-F 0 "#PWR33" H 6300 3060 30  0001 C CNN
+F 0 "#PWR063" H 6300 3060 30  0001 C CNN
 F 1 "+3.3V" H 6300 3210 30  0000 C CNN
 F 2 "" H 6300 3100 60  0000 C CNN
@@
 $EndComp
 $Comp
-L C C18
+L C C19
 U 1 1 5550B925
 P 4450 3900
-F 0 "C18" H 4450 4000 40  0000 L CNN
+F 0 "C19" H 4450 4000 40  0000 L CNN
 F 1 "10nf" H 4456 3815 40  0000 L CNN
 F 2 "Capacitors_SMD:C_0402" H 4488 3750 30  0001 C CNN
@@
 $EndComp
 $Comp
-L C C19
+L C C20
 U 1 1 5550B993
 P 4450 4150
-F 0 "C19" H 4450 4250 40  0000 L CNN
+F 0 "C20" H 4450 4250 40  0000 L CNN
 F 1 "1nf" H 4456 4065 40  0000 L CNN
 F 2 "Capacitors_SMD:C_0402" H 4488 4000 30  0001 C CNN
@@
 $EndComp
 $Comp
-L GND #PWR27
+L GND #PWR064
 U 1 1 5550B9EE
 P 4000 4300
-F 0 "#PWR27" H 4000 4300 30  0001 C CNN
+F 0 "#PWR064" H 4000 4300 30  0001 C CNN
 F 1 "GND" H 4000 4230 30  0001 C CNN
 F 2 "" H 4000 4300 60  0000 C CNN
@@
 PAInput
 $Comp
-L C C30
+L C C31
 U 1 1 5550D339
 P 7300 4650
-F 0 "C30" H 7300 4750 40  0000 L CNN
+F 0 "C31" H 7300 4750 40  0000 L CNN
 F 1 "33pf" H 7306 4565 40  0000 L CNN
 F 2 "Capacitors_SMD:C_0402" H 7338 4500 30  0001 C CNN
@@
 $EndComp
 $Comp
-L C C33
+L C C35
 U 1 1 5550D5C9
 P 8250 3250
-F 0 "C33" H 8250 3350 40  0000 L CNN
+F 0 "C35" H 8250 3350 40  0000 L CNN
 F 1 "1nf" H 8256 3165 40  0000 L CNN
 F 2 "Capacitors_SMD:C_0402" H 8288 3100 30  0001 C CNN
@@
 $EndComp
 $Comp
-L C C32
+L C C34
 U 1 1 5550D613
 P 8250 3000
-F 0 "C32" H 8250 3100 40  0000 L CNN
+F 0 "C34" H 8250 3100 40  0000 L CNN
 F 1 "3.3uf" H 8256 2915 40  0000 L CNN
 F 2 "Capacitors_SMD:C_1206" H 8288 2850 30  0001 C CNN
@@
 $EndComp
 $Comp
-L C C34
+L C C36
 U 1 1 5550D690
 P 9000 4250
-F 0 "C34" H 9000 4350 40  0000 L CNN
+F 0 "C36" H 9000 4350 40  0000 L CNN
 F 1 "56pf" H 9006 4165 40  0000 L CNN
 F 2 "Capacitors_SMD:C_0402" H 9038 4100 30  0001 C CNN
@@
 $EndComp
 $Comp
-L C C35
+L C C37
 U 1 1 5550D6DB
 P 9350 3950
-F 0 "C35" H 9350 4050 40  0000 L CNN
+F 0 "C37" H 9350 4050 40  0000 L CNN
 F 1 "100pf" H 9356 3865 40  0000 L CNN
 F 2 "Capacitors_SMD:C_0402" H 9388 3800 30  0001 C CNN
@@
 $EndComp
 $Comp
-L GND #PWR36
+L GND #PWR065
 U 1 1 5550EACC
 P 7300 5100
-F 0 "#PWR36" H 7300 5100 30  0001 C CNN
+F 0 "#PWR065" H 7300 5100 30  0001 C CNN
 F 1 "GND" H 7300 5030 30  0001 C CNN
 F 2 "" H 7300 5100 60  0000 C CNN
@@
 $EndComp
 $Comp
-L GND #PWR38
+L GND #PWR066
 U 1 1 5550EB01
 P 9000 4700
-F 0 "#PWR38" H 9000 4700 30  0001 C CNN
+F 0 "#PWR066" H 9000 4700 30  0001 C CNN
 F 1 "GND" H 9000 4630 30  0001 C CNN
 F 2 "" H 9000 4700 60  0000 C CNN
@@
 $EndComp
 $Comp
-L GND #PWR37
+L GND #PWR067
 U 1 1 5550EB36
 P 8550 3450
-F 0 "#PWR37" H 8550 3450 30  0001 C CNN
+F 0 "#PWR067" H 8550 3450 30  0001 C CNN
 F 1 "GND" H 8550 3380 30  0001 C CNN
 F 2 "" H 8550 3450 60  0000 C CNN
@@
 $EndComp
 $Comp
-L GND #PWR32
+L GND #PWR068
 U 1 1 5550EB6B
 P 6250 5150
-F 0 "#PWR32" H 6250 5150 30  0001 C CNN
+F 0 "#PWR068" H 6250 5150 30  0001 C CNN
 F 1 "GND" H 6250 5080 30  0001 C CNN
 F 2 "" H 6250 5150 60  0000 C CNN
@@
 NoConn ~ 5200 4250
 $Comp
-L C C37
+L C C33
 U 1 1 55F187F6
 P 8250 2750
-F 0 "C37" H 8250 2850 40  0000 L CNN
+F 0 "C33" H 8250 2850 40  0000 L CNN
 F 1 "C" H 8256 2665 40  0000 L CNN
-F 2 "" H 8288 2600 30  0000 C CNN
+F 2 "Capacitors_SMD:C_0402" H 8288 2600 30  0001 C CNN
 F 3 "" H 8250 2750 60  0000 C CNN
 	1    8250 2750
