File: hardwareRev1/Radio/radio.kicad_pcb (KiCad board)
At the start: 4 copper layers, 40.9 x 25.1 mm, 87 parts, among them J1 edgeMountSMA, J2 edgeMountSMA, P1 CONN_11X2, P2 CONN_1, P3 CONN_8, P4 CONN_5X2, P5 CONN_1, P6 CONN_1, U1 AX503, U2 PE42424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

Commit message: Made the PCB better. Need to submit for testing.
Routing:
- net GND: track 298.4 -> 315.1 mm, vias 30 -> 34
- net /SWD_CLK: track 18.5 -> 16.1 mm
- net (no net): track 0.40 -> 2.60 mm, vias 0 -> 1
- net /USBV1: track 61.5 -> 61.6 mm, vias 3 -> 1
Other:
- net class Default: via_drill 0.2 -> 0.2794
- rule trace_min: 0.1524 -> 0.006
- rule via_min_drill: 0.2 -> 0.254
- rule via_min_size: 0.5 -> 0.018
