File: hardwareRev1/Radio/radio.kicad_pcb (KiCad board)
At the start: 4 copper layers, 40.9 x 25.1 mm, 89 parts, among them J1 edgeMountSMA, J2 edgeMountSMA, P1 CONN_11X2, P2 CONN_1, P3 CONN_8, P4 CONN_5X2, P5 CONN_1, P6 CONN_1, U1 AX503, U2 PE42424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

Commit message: Finished up board and commited.
Parts:
- added REF**: MountingHole_2-5mm, hardwareRev1:MountingHole_.75mm, F.Cu at (64.5, 54.6)
- added REF**: MountingHole_2-5mm, hardwareRev1:MountingHole_.75mm, F.Cu at (67.8, 75.5)
- added REF**: MountingHole_2-5mm, hardwareRev1:MountingHole_.75mm, F.Cu at (93.0, 73.7)
Routing:
- net GND: track 317.0 -> 314.8 mm
- net /USBV1: track 61.5 -> 62.5 mm
- net /CLK: track 32.8 -> 32.0 mm
Other:
- board size 40.9 x 25.1 mm -> 40.9 x 24.9 mm
- board text added: "AB1TJ APRSDongle"
- board text added: "CLK"
- board text added: "DIO"
- board text added: "Exsisto nimis piger deficere."
- board text added: "GPS->"
- board text added: "REV2"
- board text added: "RF->"
- board text added: "RST"
