File: hardwareRev1/power/power.sch (KiCad schematic (older format))
At the start: 25 parts, among them IC1 ATTINY24A-M-FIXED, P1 VIN, P2 CONN_11X2, P3 AVRProg, U1 TPS63020, U2 NCP508

Commit message: added the power board.
Parts:
- C1: footprint (none) -> Capacitors_SMD:C_0201
- C2: footprint (none) -> Capacitors_SMD:c_elec_5x5.8
- C3, C4, C5: footprint (none) -> Capacitors_SMD:C_0603
- C6: footprint (none) -> Capacitors_SMD:c_elec_6.3x7.7
- D1: footprint (none) -> Diodes_SMD:SOD-323
- D2, D3: footprint (none) -> LEDs:LED-0805
- F1: footprint (none) -> SMD_Packages:SMD-2112_Pol
- IC1: footprint QFN/MLF20 -> Housings_DFN_QFN:QFN-20-1EP_4x4mm_Pitch0.5mm
- L1: footprint (none) -> Inductors:SELF-WE-TPC_M
- P1: footprint (none) -> Pin_Headers:Pin_Header_Straight_1x02
- P2: footprint (none) -> Pin_Headers:Pin_Header_Straight_2x11
- P3: footprint (none) -> Pin_Headers:Pin_Header_Straight_2x03
- R1, R2, R3, R4, R5, R6, R7: footprint (none) -> Resistors_SMD:R_0603
- TP1: footprint SparkFun-PAD.02X.02 -> Measurement_Points:Measurement_Point_Round-SMD-Pad_Big
- U1: footprint (none) -> TPS63020:TPS63020
- U2: footprint (none) -> SMD:SOT-23-5
Changed lines of the file:
@@
 F 0 "P2" H 1750 1950 60  0000 C CNN
 F 1 "CONN_11X2" V 1750 1300 50  0000 C CNN
-F 2 "" H 1750 1400 60  0000 C CNN
+F 2 "Pin_Headers:Pin_Header_Straight_2x11" H 1750 1400 60  0001 C CNN
 F 3 "" H 1750 1400 60  0000 C CNN
 	1    1750 1400
@@
 F 0 "U1" H 3950 4650 60  0000 C CNN
 F 1 "TPS63020" H 3950 4500 60  0000 C CNN
-F 2 "" H 3900 4250 60  0000 C CNN
+F 2 "TPS63020:TPS63020" H 3900 4250 60  0001 C CNN
 F 3 "" H 3900 4250 60  0000 C CNN
 	1    3900 4250
@@
 F 0 "L1" H 3850 3200 50  0000 C CNN
 F 1 "1uh" H 3850 3050 50  0000 C CNN
-F 2 "" H 3850 3100 60  0000 C CNN
+F 2 "Inductors:SELF-WE-TPC_M" H 3850 3100 60  0001 C CNN
 F 3 "" H 3850 3100 60  0000 C CNN
 	1    3850 3100
@@
 F 0 "R3" V 5280 4150 40  0000 C CNN
 F 1 "768J" V 5207 4151 40  0000 C CNN
-F 2 "" V 5130 4150 30  0000 C CNN
+F 2 "Resistors_SMD:R_0603" V 5130 4150 30  0001 C CNN
 F 3 "" H 5200 4150 30  0000 C CNN
 	1    5200 4150
@@
 F 0 "R4" V 5280 4850 40  0000 C CNN
 F 1 "137J" V 5207 4851 40  0000 C CNN
-F 2 "" V 5130 4850 30  0000 C CNN
+F 2 "Resistors_SMD:R_0603" V 5130 4850 30  0001 C CNN
 F 3 "" H 5200 4850 30  0000 C CNN
 	1    5200 4850
@@
 F 0 "C1" H 1800 4500 40  0000 L CNN
 F 1 "10u" H 1806 4315 40  0000 L CNN
-F 2 "" H 1838 4250 30  0000 C CNN
+F 2 "Capacitors_SMD:C_0201" H 1838 4250 30  0001 C CNN
 F 3 "" H 1800 4400 60  0000 C CNN
 	1    1800 4400
@@
 F 0 "C2" H 2000 4500 40  0000 L CNN
 F 1 "10u" H 2006 4315 40  0000 L CNN
-F 2 "" H 2038 4250 30  0000 C CNN
+F 2 "Capacitors_SMD:c_elec_5x5.8" H 2038 4250 30  0001 C CNN
 F 3 "" H 2000 4400 60  0000 C CNN
 	1    2000 4400
@@
 F 0 "U2" H 5300 1600 40  0000 C CNN
 F 1 "NCP508" H 5300 1550 40  0000 C CNN
-F 2 "" H 5300 1350 60  0000 C CNN
+F 2 "SMD:SOT-23-5" H 5300 1350 60  0001 C CNN
 F 3 "" H 5300 1350 60  0000 C CNN
 	1    5300 1350
@@
 F 0 "C5" H 6050 1600 40  0000 L CNN
 F 1 "1u" H 6056 1415 40  0000 L CNN
-F 2 "" H 6088 1350 30  0000 C CNN
+F 2 "Capacitors_SMD:C_0603" H 6088 1350 30  0001 C CNN
 F 3 "" H 6050 1500 60  0000 C CNN
 	1    6050 1500
@@
 F 0 "C4" H 4400 1600 40  0000 L CNN
 F 1 "1u" H 4406 1415 40  0000 L CNN
-F 2 "" H 4438 1350 30  0000 C CNN
+F 2 "Capacitors_SMD:C_0603" H 4438 1350 30  0001 C CNN
 F 3 "" H 4400 1500 60  0000 C CNN
 	1    4400 1500
@@
 F 0 "R5" V 5730 3850 40  0000 C CNN
 F 1 "R" V 5657 3851 40  0000 C CNN
-F 2 "" V 5580 3850 30  0000 C CNN
+F 2 "Resistors_SMD:R_0603" V 5580 3850 30  0001 C CNN
 F 3 "" H 5650 3850 30  0000 C CNN
 	1    5650 3850
@@
 F 0 "R1" V 1280 4450 40  0000 C CNN
 F 1 "R" V 1207 4451 40  0000 C CNN
-F 2 "" V 1130 4450 30  0000 C CNN
+F 2 "Resistors_SMD:R_0603" V 1130 4450 30  0001 C CNN
 F 3 "" H 1200 4450 30  0000 C CNN
 	1    1200 4450
@@
 F 0 "R2" V 1280 5150 40  0000 C CNN
 F 1 "R" V 1207 5151 40  0000 C CNN
-F 2 "" V 1130 5150 30  0000 C CNN
+F 2 "Resistors_SMD:R_0603" V 1130 5150 30  0001 C CNN
 F 3 "" H 1200 5150 30  0000 C CNN
 	1    1200 5150
@@
 F 0 "P3" H 7800 1000 50  0000 C CNN
 F 1 "AVRProg" V 7800 800 40  0000 C CNN
-F 2 "" H 7800 750 60  0000 C CNN
+F 2 "Pin_Headers:Pin_Header_Straight_2x03" H 7800 750 60  0001 C CNN
 F 3 "" H 7800 750 60  0000 C CNN
 	1    7800 750
@@
 F 0 "TP1" H 3100 4900 50  0000 C CNN
 F 1 "TEST-POINT2" H 3100 4700 50  0000 C CNN
-F 2 "SparkFun-PAD.02X.02" H 3100 4600 50  0001 C CNN
+F 2 "Measurement_Points:Measurement_Point_Round-SMD-Pad_Big" H 3100 4600 50  0001 C CNN
 F 3 "" H 3050 4800 60  0000 C CNN
 	1    3050 4800
@@
 F 0 "C6" H 6200 4200 40  0000 L CNN
 F 1 "120u" H 6206 4015 40  0000 L CNN
-F 2 "" H 6238 3950 30  0000 C CNN
+F 2 "Capacitors_SMD:c_elec_6.3x7.7" H 6238 3950 30  0001 C CNN
 F 3 "" H 6200 4100 60  0000 C CNN
 	1    6200 4100
@@
 F 0 "C3" H 2250 4800 40  0000 L CNN
 F 1 "100n" H 2256 4615 40  0000 L CNN
-F 2 "" H 2288 4550 30  0000 C CNN
+F 2 "Capacitors_SMD:C_0603" H 2288 4550 30  0001 C CNN
 F 3 "" H 2250 4700 60  0000 C CNN
 	1    2250 4700
@@
 F 0 "D2" H 9900 1950 50  0000 C CNN
 F 1 "STAT1G" H 9900 1750 50  0000 C CNN
-F 2 "" H 9900 1850 60  0000 C CNN
+F 2 "LEDs:LED-0805" H 9900 1850 60  0001 C CNN
 F 3 "" H 9900 1850 60  0000 C CNN
 	1    9900 1850
@@
 F 0 "D3" H 9900 2350 50  0000 C CNN
 F 1 "STAT2R" H 9900 2150 50  0000 C CNN
-F 2 "" H 9900 2250 60  0000 C CNN
+F 2 "LEDs:LED-0805" H 9900 2250 60  0001 C CNN
 F 3 "" H 9900 2250 60  0000 C CNN
 	1    9900 2250
@@
 F 0 "P1" V 550 2800 40  0000 C CNN
 F 1 "VIN" V 650 2800 40  0000 C CNN
-F 2 "" H 600 2800 60  0000 C CNN
+F 2 "Pin_Headers:Pin_Header_Straight_1x02" H 600 2800 60  0001 C CNN
 F 3 "" H 600 2800 60  0000 C CNN
 	1    600  2800
@@
 F 0 "D1" H 1850 2900 40  0000 C CNN
 F 1 "DIODE" H 1850 2700 40  0000 C CNN
-F 2 "" H 1850 2800 60  0000 C CNN
+F 2 "Diodes_SMD:SOD-323" H 1850 2800 60  0001 C CNN
 F 3 "" H 1850 2800 60  0000 C CNN
 	1    1850 2800
@@
 F 0 "F1" H 1400 2750 40  0000 C CNN
 F 1 "FUSE" H 1200 2650 40  0000 C CNN
-F 2 "" H 1300 2700 60  0000 C CNN
+F 2 "SMD_Packages:SMD-2112_Pol" H 1300 2700 60  0001 C CNN
 F 3 "" H 1300 2700 60  0000 C CNN
 	1    1300 2700
@@
 F 0 "R6" V 10680 1850 40  0000 C CNN
 F 1 "R" V 10607 1851 40  0000 C CNN
-F 2 "" V 10530 1850 30  0000 C CNN
+F 2 "Resistors_SMD:R_0603" V 10530 1850 30  0001 C CNN
 F 3 "" H 10600 1850 30  0000 C CNN
 	1    10600 1850
@@
 F 0 "R7" V 10680 2250 40  0000 C CNN
 F 1 "75" V 10607 2251 40  0000 C CNN
-F 2 "" V 10530 2250 30  0000 C CNN
+F 2 "Resistors_SMD:R_0603" V 10530 2250 30  0001 C CNN
 F 3 "" H 10600 2250 30  0000 C CNN
 	1    10600 2250
@@
 F 0 "IC1" H 6950 2500 40  0000 C CNN
 F 1 "ATTINY24A-M-FIXED" H 8500 1000 40  0000 C CNN
-F 2 "QFN/MLF20" H 7800 1550 35  0000 C CIN
+F 2 "Housings_DFN_QFN:QFN-20-1EP_4x4mm_Pitch0.5mm" H 7800 1550 35  0000 C CIN
 F 3 "" H 7800 1750 60  0000 C CNN
 	1    7800 1750

Commit message: Finished the power supbsystem.
Parts:
- added R8, R9: 100K, Resistors_SMD:R_0603, symbol R
- C1: footprint Capacitors_SMD:C_0201 -> Capacitors_SMD:C_0805
- C2: footprint Capacitors_SMD:c_elec_5x5.8 -> Capacitors_SMD:C_0805
- D1: footprint Diodes_SMD:SOD-323 -> Diodes_ThroughHole:Diode_DO-41_SOD81_Vertical_KathodeUp
- IC1: footprint Housings_DFN_QFN:QFN-20-1EP_4x4mm_Pitch0.5mm -> w_smd_qfn:qfn-20
- P2: footprint Pin_Headers:Pin_Header_Straight_2x11 -> hardwareRev1:1.27mmPitchHeader11X2
- R3: value 768J -> 768K
- R4: value 137J -> 137K
- R5: value R -> 0.01
- R6: value R -> 55
- TP1: footprint Measurement_Points:Measurement_Point_Round-SMD-Pad_Big -> Measurement_Points:Measurement_Point_Round-SMD-Pad_Small
- U1: footprint TPS63020:TPS63020 -> hardwareRev1:TPS63020
Connections:
- net labels added: BattIn, ISenceHi, ISenceHigh
- net labels removed: VOut2
- wire segments 128 -> 137
Changed lines of the file:
@@
 F 0 "P2" H 1750 1950 60  0000 C CNN
 F 1 "CONN_11X2" V 1750 1300 50  0000 C CNN
-F 2 "Pin_Headers:Pin_Header_Straight_2x11" H 1750 1400 60  0001 C CNN
+F 2 "hardwareRev1:1.27mmPitchHeader11X2" H 1750 1400 60  0001 C CNN
 F 3 "" H 1750 1400 60  0000 C CNN
 	1    1750 1400
 	1    0    0    -1
 $EndComp
-Text Label 950  950  0    60   ~ 0
-Vin
-Text Label 950  1050 0    60   ~ 0
-VOut2
 Text Label 950  1150 0    60   ~ 0
 3v3Out
@@
 Text Label 950  1750 0    60   ~ 0
 3v3Out
-Text Label 950  1850 0    60   ~ 0
-VOut2
-Text Label 950  1950 0    60   ~ 0
-Vin
-Text Label 2300 950  0    60   ~ 0
-Vin
-Text Label 2300 1050 0    60   ~ 0
-VOut2
 Text Label 2300 1150 0    60   ~ 0
 3v3Out
@@
 Text Label 2300 1750 0    60   ~ 0
 3v3Out
-Text Label 2300 1850 0    60   ~ 0
-VOut2
-Text Label 2300 1950 0    60   ~ 0
-Vin
 $Comp
 L TPS63020 U1
@@
 F 0 "U1" H 3950 4650 60  0000 C CNN
 F 1 "TPS63020" H 3950 4500 60  0000 C CNN
-F 2 "TPS63020:TPS63020" H 3900 4250 60  0001 C CNN
+F 2 "hardwareRev1:TPS63020" H 3900 4250 60  0001 C CNN
 F 3 "" H 3900 4250 60  0000 C CNN
 	1    3900 4250
@@
 P 5200 4150
 F 0 "R3" V 5280 4150 40  0000 C CNN
-F 1 "768J" V 5207 4151 40  0000 C CNN
+F 1 "768K" V 5207 4151 40  0000 C CNN
 F 2 "Resistors_SMD:R_0603" V 5130 4150 30  0001 C CNN
 F 3 "" H 5200 4150 30  0000 C CNN
@@
 P 5200 4850
 F 0 "R4" V 5280 4850 40  0000 C CNN
-F 1 "137J" V 5207 4851 40  0000 C CNN
+F 1 "137K" V 5207 4851 40  0000 C CNN
 F 2 "Resistors_SMD:R_0603" V 5130 4850 30  0001 C CNN
 F 3 "" H 5200 4850 30  0000 C CNN
@@
 F 0 "C1" H 1800 4500 40  0000 L CNN
 F 1 "10u" H 1806 4315 40  0000 L CNN
-F 2 "Capacitors_SMD:C_0201" H 1838 4250 30  0001 C CNN
+F 2 "Capacitors_SMD:C_0805" H 1838 4250 30  0001 C CNN
 F 3 "" H 1800 4400 60  0000 C CNN
 	1    1800 4400
@@
 F 0 "C2" H 2000 4500 40  0000 L CNN
 F 1 "10u" H 2006 4315 40  0000 L CNN
-F 2 "Capacitors_SMD:c_elec_5x5.8" H 2038 4250 30  0001 C CNN
+F 2 "Capacitors_SMD:C_0805" H 2038 4250 30  0001 C CNN
 F 3 "" H 2000 4400 60  0000 C CNN
 	1    2000 4400
@@
 	8850 2350 10200 2350
 Wire Wire Line
-	3250 4700 2850 4700
+	2750 4700 3250 4700
 Wire Wire Line
 	3250 4400 2850 4400
@@
 P 5650 3850
 F 0 "R5" V 5730 3850 40  0000 C CNN
-F 1 "R" V 5657 3851 40  0000 C CNN
+F 1 "0.01" V 5657 3851 40  0000 C CNN
 F 2 "Resistors_SMD:R_0603" V 5580 3850 30  0001 C CNN
 F 3 "" H 5650 3850 30  0000 C CNN
@@
 ISense
 $Comp
-L +3.3V #PWR013
-U 1 1 55494ACE
-P 9850 1300
-F 0 "#PWR013" H 9850 1260 30  0001 C CNN
-F 1 "+3.3V" H 9850 1410 30  0000 C CNN
-F 2 "" H 9850 1300 60  0000 C CNN
-F 3 "" H 9850 1300 60  0000 C CNN
-	1    9850 1300
-	1    0    0    -1
-$EndComp
-Wire Wire Line
-	9850 1350 9850 1300
-$Comp
 L CONN_3X2 P3
 U 1 1 55494EEA
@@
 F 0 "TP1" H 3100 4900 50  0000 C CNN
 F 1 "TEST-POINT2" H 3100 4700 50  0000 C CNN
-F 2 "Measurement_Points:Measurement_Point_Round-SMD-Pad_Big" H 3100 4600 50  0001 C CNN
+F 2 "Measurement_Points:Measurement_Point_Round-SMD-Pad_Small" H 3100 4600 50  0001 C CNN
 F 3 "" H 3050 4800 60  0000 C CNN
 	1    3050 4800
@@
 $EndComp
 $Comp
-L GND #PWR014
+L GND #PWR013
 U 1 1 554968EB
 P 10850 2400
-F 0 "#PWR014" H 10850 2400 30  0001 C CNN
+F 0 "#PWR013" H 10850 2400 30  0001 C CNN
 F 1 "GND" H 10850 2330 30  0001 C CNN
 F 2 "" H 10850 2400 60  0000 C CNN
@@
 F 0 "D1" H 1850 2900 40  0000 C CNN
 F 1 "DIODE" H 1850 2700 40  0000 C CNN
-F 2 "Diodes_SMD:SOD-323" H 1850 2800 60  0001 C CNN
+F 2 "Diodes_ThroughHole:Diode_DO-41_SOD81_Vertical_KathodeUp" H 1850 2800 60  0001 C CNN
 F 3 "" H 1850 2800 60  0000 C CNN
 	1    1850 2800
@@
 $EndComp
 $Comp
-L GND #PWR015
+L GND #PWR014
 U 1 1 554974F9
 P 1850 3150
-F 0 "#PWR015" H 1850 3150 30  0001 C CNN
+F 0 "#PWR014" H 1850 3150 30  0001 C CNN
 F 1 "GND" H 1850 3080 30  0001 C CNN
 F 2 "" H 1850 3150 60  0000 C CNN
@@
 P 10600 1850
 F 0 "R6" V 10680 1850 40  0000 C CNN
-F 1 "R" V 10607 1851 40  0000 C CNN
+F 1 "55" V 10607 1851 40  0000 C CNN
 F 2 "Resistors_SMD:R_0603" V 10530 1850 30  0001 C CNN
 F 3 "" H 10600 1850 30  0000 C CNN
@@
 	0    1    1    0
 $EndComp
-Wire Wire Line
-	10850 1850 10850 2400
 $Comp
 L ATTINY24A-M-FIXED IC1
@@
 F 0 "IC1" H 6950 2500 40  0000 C CNN
 F 1 "ATTINY24A-M-FIXED" H 8500 1000 40  0000 C CNN
-F 2 "Housings_DFN_QFN:QFN-20-1EP_4x4mm_Pitch0.5mm" H 7800 1550 35  0000 C CIN
+F 2 "w_smd_qfn:qfn-20" H 7800 1550 35  0001 C CIN
 F 3 "" H 7800 1750 60  0000 C CNN
 	1    7800 1750
@@
 	6650 2250 6650 2350
 Connection ~ 6650 2350
+Text Label 8900 1350 0    60   ~ 0
+ISenceHi
+Text Label 6050 3850 0    60   ~ 0
+ISenceHigh
+Wire Wire Line
+	10850 1850 10850 2250
+Wire Wire Line
+	10850 2400 10850 2350
+Wire Wire Line
+	10850 2350 10900 2350
+Wire Wire Line
+	10900 2350 10900 2150
+Wire Wire Line
+	10900 2150 10850 2150
+Connection ~ 10850 2150
+Wire Wire Line
+	1000 2700 1000 2300
+Wire Wire Line
+	1000 2300 1450 2300
+Connection ~ 1000 2700
+Text Label 1000 2300 0    60   ~ 0
+BattIn
+Text Label 950  1950 0    60   ~ 0
+BattIn
+Text Label 1000 950  0    60   ~ 0
+BattIn
+Text Label 2300 950  0    60   ~ 0
+BattIn
+Text Label 2300 1950 0    60   ~ 0
+BattIn
+$Comp
+L R R9
+U 1 1 554AD254
+P 2750 4950
+F 0 "R9" V 2830 4950 40  0000 C CNN
+F 1 "100K" V 2757 4951 40  0000 C CNN
+F 2 "Resistors_SMD:R_0603" V 2680 4950 30  0001 C CNN
+F 3 "" H 2750 4950 30  0000 C CNN
+	1    2750 4950
+	1    0    0    -1
+$EndComp
+$Comp
+L R R8
+U 1 1 554AD2BB
+P 2600 4400
+F 0 "R8" V 2680 4400 40  0000 C CNN
+F 1 "100K" V 2607 4401 40  0000 C CNN
+F 2 "Resistors_SMD:R_0603" V 2530 4400 30  0001 C CNN
+F 3 "" H 2600 4400 30  0000 C CNN
+	1    2600 4400
+	0    1    1    0
+$EndComp
+Wire Wire Line
+	2750 5200 2750 5500
+Connection ~ 2750 5500
+Wire Wire Line
+	2350 4400 2350 2750
+Wire Wire Line
+	2350 2750 5050 2750
+Wire Wire Line
+	5050 2750 5050 3850
+Connection ~ 5050 3850
 $EndSCHEMATC

Commit message: Fixed the errors with the initial layout
- Changed the pull resistor polarity on the enable pin.
- Brought the power save pull to Vin instead of Vout. I think this is
  better. Still defaults to non power saving
- Added more ground vias that will actually stay between zone fills.
- Made the current sensing actually work. Hi != High
Should work better.
Connections:
- net labels removed: ISenceHigh
- wire segments 137 -> 135
Other:
- note added: "THis should be right. \n"
Changed lines of the file:
@@
 ISenceHi
 Text Label 6050 3850 0    60   ~ 0
-ISenceHigh
+ISenceHi
 Wire Wire Line
 	10850 1850 10850 2250
@@
 	0    1    1    0
 $EndComp
+Connection ~ 2750 5500
+Connection ~ 5050 3850
 Wire Wire Line
-	2750 5200 2750 5500
-Connection ~ 2750 5500
+	2750 5200 2400 5200
+Text Label 2400 5200 0    60   ~ 0
+Vin
 Wire Wire Line
-	2350 4400 2350 2750
-Wire Wire Line
-	2350 2750 5050 2750
-Wire Wire Line
-	5050 2750 5050 3850
-Connection ~ 5050 3850
+	2350 4400 2350 4150
+Connection ~ 2350 4150
+Text Notes 2200 4050 0    60   ~ 0
+THis should be right. \n
 $EndSCHEMATC
