File: hardware/powerRev2/_saved_dualIdealDiode.sch (KiCad schematic (older format))
At the start: 10 parts

Commit message: Made progress on the board.
Connections:
- net STAT1: no longer R?.2, U?.11 (STAT2)
- new net STAT2: R?.2, U?.11 (STAT2)
Changed lines of the file:
@@
 $EndComp
 Text HLabel 8300 3950 3    60   Input ~ 0
-STAT1
+STAT2
 Wire Wire Line
 	6950 4000 6750 4000
