File: hardware/powerRev2/powerRev2.kicad_pcb (KiCad board)
At the start: 2 copper layers, 88 parts, among them P1 12Vin, P2 TC2030-CTX, P3 CONN_8X2, P4 CONN_11X2, Q1 NPN, Q2 MOSFET_P, Q3 MOS_N, U1 KL03-QFN24, U2 NCP1117ST33T3G, U3 LT6105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

Commit message: Finished the new power board.
Parts:
- removed C1: C, Capacitors_SMD:C_0402
- added BT1: BATTERY, hardwareRev1:lifepo4-1004045-3C-folded, B.Cu at (92.7, 69.5)
- added BT2: BATTERY, Pin_Headers:Pin_Header_Straight_1x02, F.Cu at (52.4, 84.0)
- added G***: LOGO, logo:logosmall, B.Cu at (76.0, 52.0)
- added P10: 3v3Vout, ultrafit:ultraFitCONN_2, F.Cu at (89.8, 86.0)
- added P11: HOLE_1, Mounting_Holes:MountingHole_2-5mm, F.Cu at (63.0, 87.0)
- added P12: HOLE_2, Mounting_Holes:MountingHole_2-5mm, F.Cu at (63.0, 48.0)
- added P13: HOLE_3, Mounting_Holes:MountingHole_2-5mm, F.Cu at (89.0, 48.0)
- added P14: HOLE_4, Mounting_Holes:MountingHole_2-5mm, F.Cu at (76.0, 87.0)
- added P5: CONN_1, Wire_Pads:SolderWirePad_single_0-8mmDrill, F.Cu at (79.4, 73.7)
- added P6: CONN_1, Wire_Pads:SolderWirePad_single_0-8mmDrill, F.Cu at (79.7, 75.5)
- added P7: CONN_1, Wire_Pads:SolderWirePad_single_0-8mmDrill, F.Cu at (78.3, 67.4)
- added P8: CONN_1, Wire_Pads:SolderWirePad_single_0-8mmDrill, F.Cu at (77.1, 68.5)
- added P9: 12Vin2, ultrafit:ultraFitCONN_2, F.Cu at (49.9, 46.3)
- added R44: 2000, Resistors_SMD:R_0402, F.Cu at (85.5, 64.1)
- added R45: 2000, Resistors_SMD:R_0402, F.Cu at (87.7, 64.1)
- Q1: value NPN -> NPN-numbered
- Q3: value MOS_N -> MOS_N_numbered
- U2: value NCP1117ST33T3G -> TLV71209DBV; footprint SMD_Packages:SOT-223 -> Housings_SOT-23_SOT-143_TSOT-6:SOT-23-5
- moved R15 101.6 mm to (77.8, 58.9), turned to 270 degrees
- moved C2 101.6 mm to (77.2, 67.0), turned to 90 degrees
- moved C3 96.9 mm to (84.9, 68.0), turned to 90 degrees
- moved D4 87.3 mm to (76.4, 61.4), turned to 90 degrees
- moved R14 82.7 mm to (76.4, 58.9), turned to 270 degrees
- moved D5 82.2 mm to (77.7, 61.4), turned to 90 degrees
- moved R8 79.5 mm to (81.6, 61.6)
- moved R1 66.7 mm to (87.5, 57.6), turned to 270 degrees
- moved TH1 65.2 mm to (83.8, 54.1), turned to 90 degrees
- moved P2 39.2 mm to (83.0, 59.0)
- moved D8 12.1 mm to (80.0, 53.3)
- moved C14 10.8 mm to (51.2, 71.1), turned to 270 degrees
- moved R33 10.00 mm to (48.2, 73.0), turned to 90 degrees
- moved R22 9.67 mm to (67.2, 77.3), turned to 90 degrees
- moved L2 9.50 mm to (60.5, 69.3), turned to 0 degrees
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Connections:
- R38 pad 1: /dualIdealDiode/Curren1 -> /dualIdealDiode/Current1
- R39 pad 1: Net-(R39-Pad1) -> /dualIdealDiode/Current2
- U1 pad 12: /dualIdealDiode/Curren1 -> /dualIdealDiode/Current1
- U1 pad 13: /dualIdealDiode/Curren1 -> /dualIdealDiode/Current2
- U1 pad 25: (no net) -> GND
- U2 pad 1: GND -> Net-(C4-Pad1)
- U2 pad 2: Net-(C6-Pad1) -> GND
- U2 pad 4: Net-(C6-Pad1) -> (no net)
- U7 pad 4: /dualIdealDiode/Curren1 -> /dualIdealDiode/Current1
- U7 pad 5: Net-(R39-Pad1) -> /dualIdealDiode/Current2
Routing:
- net GND: track 51.4 -> 434.2 mm, vias 6 -> 85
- net /dualIdealDiode/OUT1: track 16.4 -> 71.0 mm, vias 2 -> 3
- net /I2C_SDA: track 0.00 -> 39.2 mm, vias 0 -> 1
- net /VBackup: track 1.72 -> 40.2 mm, vias 0 -> 3
- net /lifepo4Charger/FAULT: track 1.56 -> 38.7 mm, vias 1 -> 2
- net /lifepo4Charger/SHDN: track 5.98 -> 42.9 mm, vias 0 -> 4
- net /I2C_SCL: track 0.00 -> 36.9 mm, vias 0 -> 2
- net /lifepo4Charger/CHRG: track 1.37 -> 33.4 mm, vias 1 -> 2
- net /BatVOut: track 2.90 -> 34.8 mm, vias 0 -> 2
- net /IRQ: track 0.00 -> 23.5 mm, vias 0 -> 2
- net /VInSense: track 1.60 -> 23.9 mm, vias 0 -> 2
- net /SwitchVOut: track 0.00 -> 20.1 mm
- net /MainCurrent: track 1.57 -> 21.1 mm, vias 0 -> 2
- net /dualIdealDiode/EN2: track 6.36 -> 24.7 mm, vias 0 -> 2
- net /dualIdealDiode/Current2: track 0.00 -> 17.9 mm, vias 0 -> 2
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- added copper zone on B.Cu, net GND
- added copper zone on F.Cu, net GND
Other:
- board outline added: 46.3 x 47.6 mm
- net class Default: clearance 0.2 -> 0.1524; trace_width 0.25 -> 0.1524
- rule trace_clearance: 0.2 -> 0.1524
- rule trace_min: 0.2 -> 0.1524
- board text added: "1"
- board text added: "AB1TJ Power Giant Rev 2"
- board text added: "Exsisto nimis piger deficere."
- board text added: "GND VIN"
- board text added: "GND VOUT"
