File: hardware/powerRev2/powerRev2.sch (KiCad schematic (older format))
At the start: 16 parts

Commit message: More work on the new power supply
Started (finished) the lifepo4 charger.
Started on the ideal diode sheet.
Still need to add uc.
Parts:
- added R?: R, symbol R
Connections:
- wire segments 37 -> 41
Changed lines of the file:
@@
 LIBS:lt6105
 LIBS:tps563200
+LIBS:lt3652
 LIBS:powerRev2-cache
 EELAYER 25 0
@@
 $Descr A4 11693 8268
 encoding utf-8
-Sheet 1 2
+Sheet 1 3
 Title ""
 Date ""
@@
 Connection ~ 4850 2300
 Wire Wire Line
-	4850 2850 4850 3750
+	4850 2850 4850 4650
 Wire Wire Line
 	4850 2900 4950 2900
@@
 Wire Wire Line
 	5550 3950 5700 3950
+$Sheet
+S 5750 4450 950  700
+U 56114AF5
+F0 "lifepo4Charger" 60
+F1 "lifepo4Charger.sch" 60
+F2 "Vin" I L 5750 4650 60
+F3 "GND" I L 5750 4950 60
+F4 "Vout" I R 6700 4600 60
+F5 "SHDN" I R 6700 4950 60
+F6 "CHRG" I R 6700 4850 60
+F7 "FAULT" I R 6700 5050 60
+$EndSheet
+$Comp
+L R R?
+U 1 1 56129619
+P 5250 4650
+F 0 "R?" V 5330 4650 40  0000 C CNN
+F 1 "R" V 5257 4651 40  0000 C CNN
+F 2 "" V 5180 4650 30  0000 C CNN
+F 3 "" H 5250 4650 30  0000 C CNN
+	1    5250 4650
+	0    1    1    0
+$EndComp
+$Comp
+L GND #PWR?
+U 1 1 56129679
+P 5450 5050
+F 0 "#PWR?" H 5450 5050 30  0001 C CNN
+F 1 "GND" H 5450 4980 30  0001 C CNN
+F 2 "" H 5450 5050 60  0000 C CNN
+F 3 "" H 5450 5050 60  0000 C CNN
+	1    5450 5050
+	1    0    0    -1
+$EndComp
+Wire Wire Line
+	5750 4650 5500 4650
+Wire Wire Line
+	4850 4650 5000 4650
+Connection ~ 4850 3750
+Wire Wire Line
+	5750 4950 5450 4950
+Wire Wire Line
+	5450 4950 5450 5050
+$Sheet
+S 7500 3900 900  550
+U 56129ACB
+F0 "dualIdealDiode" 60
+F1 "dualIdealDiode.sch" 60
+$EndSheet
 $EndSCHEMATC

Commit message: More progress on the power supply. Added a KL03 for C&C.
Parts:
- removed D? (x2): DIODESCH, symbol DIODESCH
- added C?: 4.7uf, symbol C
- added C? (x3): C, symbol C
- added Q?: MOSFET_P, symbol MOSFET_P
- added R? (x3): 0, symbol R
- added R? (x2): 4K, symbol R
- added R? (x2): 1K, symbol R
- added R?: 1000, symbol R
- added R?: 200000, symbol R
- added R?: 10000, symbol R
- added U?: KL03-QFN24, MODULE, symbol KL03-QFN24
- added U?: NCP1117ST33T3G, symbol NCP1117ST33T3G
- added X?: CRYSTAL, symbol CRYSTAL
- R? (x2): value R -> 0
Connections:
- net labels added: 3v3Out, BatVOut, Charge, ChargerFault, ChargerShutdown, I2C_SCL, I2C_SDA, MainCurrent, ORCurrent1, ORCurrent2, OREnable1, OREnable2, ORStat1, ORStat2, ORWarn1, ORWarn2, SWD_CLK, SWD_DIO, SWD_RST, SwitchVOut, SwitcherEn, VBackup, VInSense, VREF, VinSense
- net labels removed: +3.3V
- wire segments 41 -> 122
Other:
- note added: "1000 Ohm will net .2V out per amp\n\n"
- note added: "Need to divide to get down to the 1.2V internal reference"
- moved on the sheet: D?, F?, P?, Q?, R?, U?

Commit message: More work on the power supply
Parts:
- removed X?: CRYSTAL, symbol CRYSTAL
- added C1, C2, C5: C, symbol C
- added C4: 10u, symbol C
- added C6: 10uf, symbol C
- added D4, D5: LED, symbol LED
- added P2: CONN_5X2, symbol CONN_5X2
- added R1: 1500, symbol R
- added R13, R14: R, symbol R
- added R22: 10000, symbol R
- added TH1: THERMISTOR, symbol THERMISTOR
- gave numbers to parts that had none: 32
Connections:
- wire segments 122 -> 151
- no-connect marks 0 -> 6
Other:
- note added: "NTC will vary from 3k to 20K\nNeed to go from 0 to 1.2V from 3v3.\n1.5K other R will lead to .23 to 1.1"
- moved on the sheet: R17, U2, U3

Commit message: Started the new power board PCB. Made it pretty far.
Parts:
- removed P2: CONN_5X2, symbol CONN_5X2
- added D8, D9: 1n4001, Diodes_SMD:SOD-323, symbol DIODE
- added P2: TC2030-CTX, Tag-Connect:TC2030-NL_SMALL, symbol TC2030-CTX
- added P3: CONN_8X2, hardwareRev1:1.27mm2X8, symbol CONN_8X2
- added P4: CONN_11X2, hardwareRev1:1.27mmPitchHeader11X2, symbol CONN_11X2
- C1, C2, C3, C5, C7, C8: footprint (none) -> Capacitors_SMD:C_0402
- C4: footprint (none) -> Capacitors_SMD:C_0805; Man PN (none) -> GRM21BR61E106KA73L; Manufacturer PN (none) -> GRM21BR61E106KA73L
- C6: footprint (none) -> Capacitors_SMD:C_0805; Manufacturer PN (none) -> GRM21BR61E106KA73L
- C9: footprint (none) -> Capacitors_SMD:C_0805; Manufacturer PN (none) -> CC0805ZRY5V6BB475
- D1, D2, D4, D5: footprint (none) -> LEDs:LED-0603
- D3: footprint (none) -> Diodes_SMD:SOD-323; Manufacturer PN (none) -> 1N4148WX-TP
- F1: footprint (none) -> Fuse_Holders_and_Fuses:Fuse_SMD2920; Manufacturer PN (none) -> MF-LSMF260X-2
- P1, TH1: footprint (none) -> Pin_Headers:Pin_Header_Straight_1x02
- Q1: footprint (none) -> Housings_SOT-23_SOT-143_TSOT-6:SOT-23; Manufacturer PN (none) -> MMBT3904-TP
- Q2: footprint (none) -> hardwareRev1:DMP2018LFK-7; Manufacturer PN (none) -> DMP2018LFK-7
- R1, R2, R3, R4, R5, R6: footprint (none) -> Resistors_SMD:R_0402
- R10: renamed from R9; footprint (none) -> Resistors_SMD:R_0402
- R11: renamed from R10; footprint (none) -> Resistors_SMD:R_0402
- R12: renamed from R11; footprint (none) -> Resistors_SMD:R_0402
- R13: renamed from R12; footprint (none) -> Resistors_SMD:R_0402
- R14: renamed from R13; footprint (none) -> Resistors_SMD:R_0402
- R15: renamed from R14; footprint (none) -> Resistors_SMD:R_0402
- R16: renamed from R15; footprint (none) -> Resistors_SMD:R_0402
- R17: renamed from R16; footprint (none) -> Resistors_SMD:R_0402
- R18: renamed from R17; footprint (none) -> Resistors_SMD:R_0402
- R19: renamed from R18; footprint (none) -> Resistors_SMD:R_0402
- R20: renamed from R19; footprint (none) -> Resistors_SMD:R_0402
- R21: renamed from R20; footprint (none) -> Resistors_SMD:R_0402
- R22: renamed from R21; footprint (none) -> Resistors_SMD:R_0402
- R7: footprint (none) -> Resistors_SMD:R_0805; Manufacturer PN (none) -> CRF0805-FX-R020ELF
- R8: renamed from R22; footprint (none) -> Resistors_SMD:R_0402
- R9: renamed from R8; footprint (none) -> Resistors_SMD:R_0402
- U1: footprint MODULE -> Housings_DFN_QFN:QFN-24-1EP_4x4mm_Pitch0.5mm
- U2: footprint (none) -> SMD_Packages:SOT-223
- U3: footprint (none) -> hardwareRev1:LT6105
Connections:
- net labels added: 12Vin, IRQ
- wire segments 151 -> 190
- no-connect marks 6 -> 9
Other:
- note added: "Ensure this \nis correct."
- note removed: "NTC will vary from 3k to 20K\nNeed to go from 0 to 1.2V from 3v3.\n1.5K other R will lead to .23 to 1.1"
- moved on the sheet: C6, R8

Commit message: Finished the new power board.
Parts:
- removed C1: C, Capacitors_SMD:C_0402, symbol C
- removed Q1: NPN, Housings_SOT-23_SOT-143_TSOT-6:SOT-23, symbol NPN
- removed U2: NCP1117ST33T3G, SMD_Packages:SOT-223, symbol NCP1117ST33T3G
- added P10: 3v3Vout, ultrafit:ultraFitCONN_2, symbol CONN_2
- added P5, P6, P7, P8: CONN_1, Wire_Pads:SolderWirePad_single_0-8mmDrill, symbol CONN_1
- added P9: 12Vin2, ultrafit:ultraFitCONN_2, symbol CONN_2
- added Q1: NPN-numbered, Housings_SOT-23_SOT-143_TSOT-6:SOT-23, symbol NPN-numbered
- added R44, R45: 4.7k, Resistors_SMD:R_0402, symbol R
- added U2: TLV71209DBV, Housings_SOT-23_SOT-143_TSOT-6:SOT-23-5, symbol TLV71209DBV
- C2, C3, C5: value C -> 1uf
- C7, C8: value C -> DNP
- R14, R15: value R -> 80
- R20, R21: value 4K -> 3.9K
- TH1: Manufacturer PN (none) -> NTCLE100E3103JB0
Connections:
- wire segments 190 -> 203
Other:
- note added: "Gives a factor of 0.2040816327.... ugh.\n"
Changed lines of the file:
@@
 EESchema Schematic File Version 2
+LIBS:powerRev2-rescue
 LIBS:power
 LIBS:device
@@
 LIBS:RF-Head2
 LIBS:ritli-rfhead
+LIBS:mos_n_numbered
+LIBS:npn-numbered
 LIBS:powerRev2-cache
 EELAYER 25 0
@@
 $EndComp
 $Comp
-L NPN Q1
-U 1 1 5611F09A
-P 1850 1600
-F 0 "Q1" H 1850 1450 50  0000 R CNN
-F 1 "NPN" H 1850 1750 50  0000 R CNN
-F 2 "Housings_SOT-23_SOT-143_TSOT-6:SOT-23" H 1850 1600 60  0001 C CNN
-F 3 "" H 1850 1600 60  0000 C CNN
-F 4 "MMBT3904-TP" H 1850 1600 60  0001 C CNN "Manufacturer PN"
-	1    1850 1600
-	-1   0    0    -1
-$EndComp
-$Comp
 L LED D1
 U 1 1 5611F130
@@
 L GND #PWR02
 U 1 1 5611F32C
-P 1100 1100
-F 0 "#PWR02" H 1100 1100 30  0001 C CNN
-F 1 "GND" H 1100 1030 30  0001 C CNN
-F 2 "" H 1100 1100 60  0000 C CNN
-F 3 "" H 1100 1100 60  0000 C CNN
-	1    1100 1100
+P 1100 2000
+F 0 "#PWR02" H 1100 2000 30  0001 C CNN
+F 1 "GND" H 1100 1930 30  0001 C CNN
+F 2 "" H 1100 2000 60  0000 C CNN
+F 3 "" H 1100 2000 60  0000 C CNN
+	1    1100 2000
 	1    0    0    -1
 $EndComp
@@
 F3 "EN1" I R 9050 3400 60
 F4 "EN2" I R 9050 3500 60
-F5 "Curren1" I R 9050 3200 60
+F5 "Current1" I R 9050 3200 60
 F6 "Current2" I R 9050 3300 60
 F7 "VIN2" I L 7800 3450 60
@@
 P 6850 2750
 F 0 "R20" V 6930 2750 40  0000 C CNN
-F 1 "4K" V 6857 2751 40  0000 C CNN
+F 1 "3.9K" V 6857 2751 40  0000 C CNN
 F 2 "Resistors_SMD:R_0402" V 6780 2750 30  0001 C CNN
 F 3 "" H 6850 2750 30  0000 C CNN
@@
 P 6850 3800
 F 0 "R21" V 6930 3800 40  0000 C CNN
-F 1 "4K" V 6857 3801 40  0000 C CNN
+F 1 "3.9K" V 6857 3801 40  0000 C CNN
 F 2 "Resistors_SMD:R_0402" V 6780 3800 30  0001 C CNN
 F 3 "" H 6850 3800 30  0000 C CNN
@@
 P 6600 2100
 F 0 "C7" H 6600 2200 40  0000 L CNN
-F 1 "C" H 6606 2015 40  0000 L CNN
+F 1 "DNP" H 6606 2015 40  0000 L CNN
 F 2 "Capacitors_SMD:C_0402" H 6638 1950 30  0001 C CNN
 F 3 "" H 6600 2100 60  0000 C CNN
@@
 P 6650 4500
 F 0 "C8" H 6650 4600 40  0000 L CNN
-F 1 "C" H 6656 4415 40  0000 L CNN
+F 1 "DNP" H 6656 4415 40  0000 L CNN
 F 2 "Capacitors_SMD:C_0402" H 6688 4350 30  0001 C CNN
 F 3 "" H 6650 4500 60  0000 C CNN
@@
 $EndComp
 $Comp
-L NCP1117ST33T3G U2
-U 1 1 561EB20E
-P 5050 800
-F 0 "U2" H 5050 1050 40  0000 C CNN
-F 1 "NCP1117ST33T3G" H 5050 1000 40  0000 C CNN
-F 2 "SMD_Packages:SOT-223" H 5050 800 60  0001 C CNN
-F 3 "" H 5050 800 60  0000 C CNN
-	1    5050 800
-	1    0    0    -1
-$EndComp
-$Comp
 L GND #PWR012
 U 1 1 561EBA89
-P 5050 1150
-F 0 "#PWR012" H 5050 1150 30  0001 C CNN
-F 1 "GND" H 5050 1080 30  0001 C CNN
-F 2 "" H 5050 1150 60  0000 C CNN
-F 3 "" H 5050 1150 60  0000 C CNN
-	1    5050 1150
+P 4950 1150
+F 0 "#PWR012" H 4950 1150 30  0001 C CNN
+F 1 "GND" H 4950 1080 30  0001 C CNN
+F 2 "" H 4950 1150 60  0000 C CNN
+F 3 "" H 4950 1150 60  0000 C CNN
+	1    4950 1150
 	1    0    0    -1
 $EndComp
@@
 P 4150 5750
 F 0 "C3" H 4150 5850 40  0000 L CNN
-F 1 "C" H 4156 5665 40  0000 L CNN
+F 1 "1uf" H 4156 5665 40  0000 L CNN
 F 2 "Capacitors_SMD:C_0402" H 4188 5600 30  0001 C CNN
 F 3 "" H 4150 5750 60  0000 C CNN
@@
 Text Label 1050 6050 0    60   ~ 0
 MainCurrent
+Text Label 3450 5950 0    60   ~ 0
+ORCurrent1
 Text Label 3450 5850 0    60   ~ 0
-ORCurrent1
-Text Label 3450 5950 0    60   ~ 0
 ORCurrent2
 Text Label 3450 5550 0    60   ~ 0
@@
 P 4900 6050
 F 0 "R14" V 4980 6050 40  0000 C CNN
-F 1 "R" V 4907 6051 40  0000 C CNN
+F 1 "80" V 4907 6051 40  0000 C CNN
 F 2 "Resistors_SMD:R_0402" V 4830 6050 30  0001 C CNN
 F 3 "" H 4900 6050 30  0000 C CNN
@@
 P 4900 6350
 F 0 "R15" V 4980 6350 40  0000 C CNN
-F 1 "R" V 4907 6351 40  0000 C CNN
+F 1 "80" V 4907 6351 40  0000 C CNN
 F 2 "Resistors_SMD:R_0402" V 4830 6350 30  0001 C CNN
 F 3 "" H 4900 6350 30  0000 C CNN
@@
 F 2 "Pin_Headers:Pin_Header_Straight_1x02" H 750 6600 60  0001 C CNN
 F 3 "" H 750 6600 60  0000 C CNN
-F 4 "NTCLE100E3103JB0" V 750 6600 60  0001 C CNN "ManPN"
+F 4 "NTCLE100E3103JB0" H 750 6600 60  0001 C CNN "Manufacturer PN"
+F 5 "NTCLE100E3103JB0" V 750 6600 60  0001 C CNN "ManPN"
 	1    750  6600
 	1    0    0    -1
@@
 P 2150 4450
 F 0 "C2" H 2150 4550 40  0000 L CNN
-F 1 "C" H 2156 4365 40  0000 L CNN
+F 1 "1uf" H 2156 4365 40  0000 L CNN
 F 2 "Capacitors_SMD:C_0402" H 2188 4300 30  0001 C CNN
 F 3 "" H 2150 4450 60  0000 C CNN
 	1    2150 4450
-	1    0    0    -1
-$EndComp
-$Comp
-L C C1
-U 1 1 56272392
-P 1900 4450
-F 0 "C1" H 1900 4550 40  0000 L CNN
-F 1 "C" H 1906 4365 40  0000 L CNN
-F 2 "Capacitors_SMD:C_0402" H 1938 4300 30  0001 C CNN
-F 3 "" H 1900 4450 60  0000 C CNN
-	1    1900 4450
 	1    0    0    -1
 $EndComp
@@
 P 4300 2000
 F 0 "C5" H 4300 2100 40  0000 L CNN
-F 1 "C" H 4306 1915 40  0000 L CNN
+F 1 "1uf" H 4306 1915 40  0000 L CNN
 F 2 "Capacitors_SMD:C_0402" H 4338 1850 30  0001 C CNN
 F 3 "" H 4300 2000 60  0000 C CNN
@@
 	1750 1800 1750 2250
 Wire Wire Line
-	1100 1100 1100 950
+	1100 950  1100 2000
 Wire Wire Line
 	1100 950  1050 950
@@
 Connection ~ 3550 750
 Wire Wire Line
-	5050 1050 5050 1150
-Wire Wire Line
 	3300 750  3650 750
-Wire Wire Line
-	4150 750  4650 750
 Wire Wire Line
 	2500 4850 2500 4700
@@
 Wire Wire Line
 	1450 600  1950 600
-Wire Wire Line
-	5450 850  5550 850
-Wire Wire Line
-	5550 850  5550 750
-Connection ~ 5550 750
 Wire Wire Line
 	5150 2200 4550 2200
@@
 $EndComp
 Wire Wire Line
-	5450 750  5800 750
+	5400 750  5800 750
 Wire Wire Line
 	5800 600  5800 900
@@
 Text Label 7550 600  0    60   ~ 0
 3v3Out
+$Comp
+L NPN-numbered Q1
+U 1 1 562FF133
+P 1850 1600
+F 0 "Q1" H 1850 1450 50  0000 R CNN
+F 1 "NPN-numbered" H 1850 1750 50  0000 R CNN
+F 2 "Housings_SOT-23_SOT-143_TSOT-6:SOT-23" H 1850 1600 60  0001 C CNN
+F 3 "" H 1850 1600 60  0000 C CNN
+F 4 "MMBT3904LT1G" H 1850 1600 60  0001 C CNN "Manufacturer PN"
+	1    1850 1600
+	-1   0    0    -1
+$EndComp
+$Comp
+L TLV71209DBV U2
+U 1 1 563003D7
+P 4950 800
+F 0 "U2" H 4700 1000 40  0000 C CNN
+F 1 "TLV71209DBV" H 5150 1000 40  0000 C CNN
+F 2 "Housings_SOT-23_SOT-143_TSOT-6:SOT-23-5" H 4950 900 35  0000 C CIN
+F 3 "" H 4950 800 60  0000 C CNN
+F 4 "AP2204K-3.3TRG1" H 4950 800 60  0001 C CNN "Manufacturer PN"
+	1    4950 800
+	1    0    0    -1
+$EndComp
+Wire Wire Line
+	4950 1100 4950 1150
+Wire Wire Line
+	4150 750  4500 750
+Wire Wire Line
+	4500 900  4400 900
+Wire Wire Line
+	4400 900  4400 750
+Connection ~ 4400 750
+Text Label 7150 6750 0    60   ~ 0
+I2C_SCL
+Text Label 7150 6950 0    60   ~ 0
+I2C_SDA
+Wire Wire Line
+	7050 6750 7600 6750
+Wire Wire Line
+	7050 6950 7600 6950
+$Comp
+L R R44
+U 1 1 56313889
+P 7850 6750
+F 0 "R44" V 7930 6750 40  0000 C CNN
+F 1 "4.7k" V 7857 6751 40  0000 C CNN
+F 2 "Resistors_SMD:R_0402" V 7780 6750 30  0001 C CNN
+F 3 "" H 7850 6750 30  0000 C CNN
+	1    7850 6750
+	0    1    1    0
+$EndComp
+$Comp
+L R R45
+U 1 1 563139B5
+P 7850 6950
+F 0 "R45" V 7930 6950 40  0000 C CNN
+F 1 "4.7k" V 7857 6951 40  0000 C CNN
+F 2 "Resistors_SMD:R_0402" V 7780 6950 30  0001 C CNN
+F 3 "" H 7850 6950 30  0000 C CNN
+	1    7850 6950
+	0    1    1    0
+$EndComp
+Wire Wire Line
+	8100 6750 8800 6750
+Wire Wire Line
+	8350 6750 8350 6950
+Wire Wire Line
+	8350 6950 8100 6950
+Connection ~ 8350 6750
+Text Label 8450 6750 0    60   ~ 0
+VBackup
+Wire Wire Line
+	2650 6850 2650 6900
+Wire Wire Line
+	2650 6900 2500 6900
+Connection ~ 2500 6900
+$Comp
+L CONN_1 P5
+U 1 1 56324297
+P 9550 3800
+F 0 "P5" H 9630 3800 40  0000 L CNN
+F 1 "CONN_1" H 9550 3855 30  0001 C CNN
+F 2 "Wire_Pads:SolderWirePad_single_0-8mmDrill" H 9550 3800 60  0001 C CNN
+F 3 "" H 9550 3800 60  0000 C CNN
+	1    9550 3800
+	1    0    0    -1
+$EndComp
+$Comp
+L CONN_1 P6
+U 1 1 5632438C
+P 9550 3900
+F 0 "P6" H 9630 3900 40  0000 L CNN
+F 1 "CONN_1" H 9550 3955 30  0001 C CNN
+F 2 "Wire_Pads:SolderWirePad_single_0-8mmDrill" H 9550 3900 60  0001 C CNN
+F 3 "" H 9550 3900 60  0000 C CNN
+	1    9550 3900
+	1    0    0    -1
+$EndComp
+$Comp
+L CONN_1 P7
+U 1 1 56326EC3
+P 900 5350
+F 0 "P7" H 980 5350 40  0000 L CNN
+F 1 "CONN_1" H 900 5405 30  0001 C CNN
+F 2 "Wire_Pads:SolderWirePad_single_0-8mmDrill" H 900 5350 60  0001 C CNN
+F 3 "" H 900 5350 60  0000 C CNN
+	1    900  5350
+	-1   0    0    1
+$EndComp
+$Comp
+L CONN_1 P8
+U 1 1 56326EC9
+P 900 5450
+F 0 "P8" H 980 5450 40  0000 L CNN
+F 1 "CONN_1" H 900 5505 30  0001 C CNN
+F 2 "Wire_Pads:SolderWirePad_single_0-8mmDrill" H 900 5450 60  0001 C CNN
+F 3 "" H 900 5450 60  0000 C CNN
+	1    900  5450
+	-1   0    0    1
+$EndComp
+$Comp
+L CONN_2 P9
+U 1 1 5640B5DF
+P 700 1550
+F 0 "P9" V 650 1550 40  0000 C CNN
+F 1 "12Vin2" V 750 1550 40  0000 C CNN
+F 2 "ultrafit:ultraFitCONN_2" H 700 1550 60  0001 C CNN
+F 3 "" H 700 1550 60  0000 C CNN
+	1    700  1550
+	-1   0    0    1
+$EndComp
+Wire Wire Line
+	1050 1650 1100 1650
+Connection ~ 1100 1650
+Wire Wire Line
+	1050 1450 1250 1450
+Wire Wire Line
+	1250 1450 1250 750
+Connection ~ 1250 750
+$Comp
+L CONN_2 P10
+U 1 1 5640CDA4
+P 10450 6850
+F 0 "P10" V 10400 6850 40  0000 C CNN
+F 1 "3v3Vout" V 10500 6850 40  0000 C CNN
+F 2 "ultrafit:ultraFitCONN_2" H 10450 6850 60  0001 C CNN
+F 3 "" H 10450 6850 60  0000 C CNN
+	1    10450 6850
+	1    0    0    -1
+$EndComp
+Text Label 9650 6750 0    60   ~ 0
+3v3Out
+Wire Wire Line
+	9550 6750 10100 6750
+$Comp
+L GND #PWR026
+U 1 1 5640DED6
+P 9950 7150
+F 0 "#PWR026" H 9950 7150 30  0001 C CNN
+F 1 "GND" H 9950 7080 30  0001 C CNN
+F 2 "" H 9950 7150 60  0000 C CNN
+F 3 "" H 9950 7150 60  0000 C CNN
+	1    9950 7150
+	1    0    0    -1
+$EndComp
+Wire Wire Line
+	10100 6950 9950 6950
+Wire Wire Line
+	9950 6950 9950 7150
+Text Notes 7000 2550 0    60   ~ 0
+Gives a factor of 0.2040816327.... ugh.\n
 $EndSCHEMATC

Commit message: Really really large commit because I like to live dangerously...
Parts:
- C2, C3, C4, C5, C6, C7, C8, C9: symbol C -> C-RESCUE-powerRev2
- D1, D2, D4, D5: symbol LED -> LED-RESCUE-powerRev2
- R1, R10, R11, R12, R13, R14, R15, R16, R17, R18, R19, R2, R20, R21, R22, R3, R4, R44, R45, R5, R6, R7, R8, R9: symbol R -> R-RESCUE-powerRev2
Changed lines of the file:
@@
 LIBS:hardwareRev1-cache
 LIBS:Tag-Connect
-LIBS:mpcie
 LIBS:RF-Head2
 LIBS:ritli-rfhead
@@
 $EndComp
 $Comp
-L R R2
+L R-RESCUE-powerRev2 R2
 U 1 1 5611F06D
 P 1450 1050
@@
 $EndComp
 $Comp
-L LED D1
+L LED-RESCUE-powerRev2 D1
 U 1 1 5611F130
 P 1450 1650
@@
 $EndComp
 $Comp
-L R R3
+L R-RESCUE-powerRev2 R3
 U 1 1 5611F154
 P 2400 1600
@@
 $EndComp
 $Comp
-L R R4
+L R-RESCUE-powerRev2 R4
 U 1 1 5611F181
 P 2700 1900
@@
 $EndComp
 $Comp
-L GND #PWR01
+L GND-RESCUE-powerRev2 #PWR01
 U 1 1 5611F2F3
 P 1900 2350
@@
 $EndComp
 $Comp
-L GND #PWR02
+L GND-RESCUE-powerRev2 #PWR02
 U 1 1 5611F32C
 P 1100 2000
@@
 $EndComp
 $Comp
-L LED D2
+L LED-RESCUE-powerRev2 D2
 U 1 1 5611F404
 P 2500 2250
@@
 $EndComp
 $Comp
-L R R7
+L R-RESCUE-powerRev2 R7
 U 1 1 5611F668
 P 3550 1700
@@
 $EndComp
 $Comp
-L R R10
+L R-RESCUE-powerRev2 R10
 U 1 1 5611F6A4
 P 3900 1400
@@
 $EndComp
 $Comp
-L R R11
+L R-RESCUE-powerRev2 R11
 U 1 1 5611F705
 P 3900 2000
@@
 $EndComp
 $Comp
-L R R12
+L R-RESCUE-powerRev2 R12
 U 1 1 5611FAFB
 P 3900 2850
@@
 $EndSheet
 $Comp
-L GND #PWR03
+L GND-RESCUE-powerRev2 #PWR03
 U 1 1 56120AF0
 P 4250 3100
@@
 $EndSheet
 $Comp
-L R R13
+L R-RESCUE-powerRev2 R13
 U 1 1 56129619
 P 3950 3750
@@
 $EndComp
 $Comp
-L GND #PWR04
+L GND-RESCUE-powerRev2 #PWR04
 U 1 1 56129679
 P 4150 4150
@@
 $EndSheet
 $Comp
-L R R16
+L R-RESCUE-powerRev2 R16
 U 1 1 5618B875
 P 5600 2800
@@
 $EndComp
 $Comp
-L R R17
+L R-RESCUE-powerRev2 R17
 U 1 1 5618BAC8
 P 5700 3700
@@
 $EndComp
 $Comp
-L GND #PWR05
+L GND-RESCUE-powerRev2 #PWR05
 U 1 1 5618C4AB
 P 7600 4100
@@
 $EndComp
 $Comp
-L C C9
+L C-RESCUE-powerRev2 C9
 U 1 1 5618C74A
 P 9300 4450
@@
 $EndComp
 $Comp
-L GND #PWR06
+L GND-RESCUE-powerRev2 #PWR06
 U 1 1 5618C7CC
 P 9300 4750
@@
 $EndComp
 $Comp
-L GND #PWR07
+L GND-RESCUE-powerRev2 #PWR07
 U 1 1 561930DF
 P 3100 1200
@@
 $EndComp
 $Comp
-L R R20
+L R-RESCUE-powerRev2 R20
 U 1 1 561DE9D7
 P 6850 2750
@@
 $EndComp
 $Comp
-L R R19
+L R-RESCUE-powerRev2 R19
 U 1 1 561DEA56
 P 6850 2100
@@
 $EndComp
 $Comp
-L R R21
+L R-RESCUE-powerRev2 R21
 U 1 1 561DEAD2
 P 6850 3800
@@
 $EndComp
 $Comp
-L R R22
+L R-RESCUE-powerRev2 R22
 U 1 1 561DEB49
 P 6850 4450
@@
 $EndComp
 $Comp
-L GND #PWR08
+L GND-RESCUE-powerRev2 #PWR08
 U 1 1 561DEBDF
 P 6850 4800
@@
 $EndComp
 $Comp
-L GND #PWR09
+L GND-RESCUE-powerRev2 #PWR09
 U 1 1 561DEC52
 P 7150 1900
@@
 MainCurrent
 $Comp
-L GND #PWR010
+L GND-RESCUE-powerRev2 #PWR010
 U 1 1 5611F90E
 P 4550 2300
@@
 Need to divide to get down to the 1.2V internal reference
 $Comp
-L R R18
+L R-RESCUE-powerRev2 R18
 U 1 1 561DF7D0
 P 5750 1950
@@
 $EndComp
 $Comp
-L GND #PWR011
+L GND-RESCUE-powerRev2 #PWR011
 U 1 1 561DFA4D
 P 5750 2300
@@
 1000 Ohm will net .2V out per amp\n\n
 $Comp
-L C C7
+L C-RESCUE-powerRev2 C7
 U 1 1 561E03A1
 P 6600 2100
@@
 SwitchVOut
 $Comp
-L C C8
+L C-RESCUE-powerRev2 C8
 U 1 1 561E0A13
 P 6650 4500
@@
 $EndComp
 $Comp
-L GND #PWR012
+L GND-RESCUE-powerRev2 #PWR012
 U 1 1 561EBA89
 P 4950 1150
@@
 VBackup
 $Comp
-L R R9
+L R-RESCUE-powerRev2 R9
 U 1 1 561EC5CA
 P 3900 750
@@
 VBackup
 $Comp
-L GND #PWR013
+L GND-RESCUE-powerRev2 #PWR013
 U 1 1 561ED290
 P 2500 6950
@@
 $EndComp
 $Comp
-L R R5
+L R-RESCUE-powerRev2 R5
 U 1 1 561EE1AC
 P 3200 2750
@@
 $EndComp
 $Comp
-L R R6
+L R-RESCUE-powerRev2 R6
 U 1 1 561EE22D
 P 3200 3350
@@
 $EndComp
 $Comp
-L GND #PWR014
+L GND-RESCUE-powerRev2 #PWR014
 U 1 1 561EE2B7
 P 3200 3700
@@
 SWD_CLK
 $Comp
-L C C3
+L C-RESCUE-powerRev2 C3
 U 1 1 561F0D2D
 P 4150 5750
@@
 $EndComp
 $Comp
-L GND #PWR015
+L GND-RESCUE-powerRev2 #PWR015
 U 1 1 561F0F52
 P 4450 5800
@@
 ChargerShutdown
 $Comp
-L LED D4
+L LED-RESCUE-powerRev2 D4
 U 1 1 5626EFCC
 P 4350 6050
@@
 $EndComp
 $Comp
-L LED D5
+L LED-RESCUE-powerRev2 D5
 U 1 1 5626F16B
 P 4350 6350
@@
 $EndComp
 $Comp
-L R R14
+L R-RESCUE-powerRev2 R14
 U 1 1 5626F3CC
 P 4900 6050
@@
 $EndComp
 $Comp
-L R R15
+L R-RESCUE-powerRev2 R15
 U 1 1 5626F457
 P 4900 6350
@@
 $EndComp
 $Comp
-L GND #PWR016
+L GND-RESCUE-powerRev2 #PWR016
 U 1 1 5626F4E9
 P 5250 6500
@@
 $EndComp
 $Comp
-L R R1
+L R-RESCUE-powerRev2 R1
 U 1 1 56270E41
 P 750 7200
@@
 $EndComp
 $Comp
-L GND #PWR017
+L GND-RESCUE-powerRev2 #PWR017
 U 1 1 56270ED3
 P 750 7600
@@
 $EndComp
 $Comp
-L C C2
+L C-RESCUE-powerRev2 C2
 U 1 1 562722CF
 P 2150 4450
@@
 $EndComp
 $Comp
-L C C4
+L C-RESCUE-powerRev2 C4
 U 1 1 562726B5
 P 4200 1000
@@
 $EndComp
 $Comp
-L C C6
+L C-RESCUE-powerRev2 C6
 U 1 1 56272A4D
 P 6150 900
@@
 $EndComp
 $Comp
-L C C5
+L C-RESCUE-powerRev2 C5
 U 1 1 56273373
 P 4300 2000
@@
 $EndComp
 $Comp
-L GND #PWR018
+L GND-RESCUE-powerRev2 #PWR018
 U 1 1 562757A3
 P 1600 4300
@@
 $EndComp
 $Comp
-L GND #PWR019
+L GND-RESCUE-powerRev2 #PWR019
 U 1 1 56276462
 P 4200 1250
@@
 $EndComp
 $Comp
-L GND #PWR020
+L GND-RESCUE-powerRev2 #PWR020
 U 1 1 56276951
 P 6400 900
@@
 SWD_RST
 $Comp
-L GND #PWR021
+L GND-RESCUE-powerRev2 #PWR021
 U 1 1 5627AD26
 P 4300 5100
@@
 $EndComp
 $Comp
-L R R8
+L R-RESCUE-powerRev2 R8
 U 1 1 5627B49C
 P 3700 4950
@@
 I2C_SDA
 $Comp
-L GND #PWR022
+L GND-RESCUE-powerRev2 #PWR022
 U 1 1 5629CB4D
 P 5600 6200
@@
 $EndComp
 $Comp
-L GND #PWR023
+L GND-RESCUE-powerRev2 #PWR023
 U 1 1 5629CD39
 P 7900 6200
@@
 3v3Out
 $Comp
-L GND #PWR024
+L GND-RESCUE-powerRev2 #PWR024
 U 1 1 562A04B5
 P 10550 6100
@@
 $EndComp
 $Comp
-L GND #PWR025
+L GND-RESCUE-powerRev2 #PWR025
 U 1 1 562A056D
 P 8500 6050
@@
 	7050 6950 7600 6950
 $Comp
-L R R44
+L R-RESCUE-powerRev2 R44
 U 1 1 56313889
 P 7850 6750
@@
 $EndComp
 $Comp
-L R R45
+L R-RESCUE-powerRev2 R45
 U 1 1 563139B5
 P 7850 6950
@@
 	9550 6750 10100 6750
 $Comp
-L GND #PWR026
+L GND-RESCUE-powerRev2 #PWR026
 U 1 1 5640DED6
 P 9950 7150
