File: hardware/Radio/_autosave-radio.kicad_pcb (KiCad board)
At the start: 4 copper layers, 40.9 x 24.9 mm, 93 parts, among them J1 edgeMountSMA, J2 edgeMountSMA, P1 CONN_11X2, P2 CONN_1, P3 CONN_8, P4 CONN_5X2, P5 CONN_1, P6 CONN_1, U1 AX503, U2 PE42424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

Commit message: Really really large commit because I like to live dangerously...
Parts:
- removed Ref**: Val**, mpcie:mpcie-full-card
