File: hardware/Radio/MCU.sch (KiCad schematic (older format))
At the start: 31 parts, among them J2 edgeMountSMA, P3 CONN_8, P4 CONN_5X2, P5 GPSDM, P6 GPSDP, P7 ID, U4 MKL26Z128VLH4, U6 MICRO-B_USB

Commit message: Annotated the schematic and board
Made the numbers increase by 100, so I can just copy this in.
Parts:
- renumbered C44 to C113, C39 to C139, C40 to C140, C38 to C141, C42 to C142, C41 to C143, C43 to C144, D1 to D101, D2 to D102, J2 to J102, JMP4 to JMP101, JMP3 to JMP102, JMP2 to JMP103, L16 to L117, P3 to P102, P6 to P103, P5 to P105, P4 to P106, R4 to R102, R5 to R103, R6 to R104, R3 to R105, R2 to R106, R7 to R107, RF2 to RF102, U6 to U104, U4 to U105
Changed lines of the file:
@@
 GPSPulse
 $Comp
-L MICRO-B_USB U6
+L MICRO-B_USB U104
 U 1 1 55F4BE34
 P 7750 5300
-F 0 "U6" H 7750 5000 50  0000 C CNN
+F 0 "U104" H 7750 5000 50  0000 C CNN
 F 1 "MICRO-B_USB" H 7750 5600 50  0000 C CNN
 F 2 "USB:USB micro B female" H 7750 5300 60  0001 C CNN
@@
 $EndComp
 $Comp
-L SJMPOpen JMP3
+L SJMPOpen JMP102
 U 1 1 55F4BE35
 P 6700 5450
-F 0 "JMP3" H 6900 5600 50  0000 C CNN
+F 0 "JMP102" H 6900 5600 50  0000 C CNN
 F 1 "SJMPOpen" H 6800 5301 40  0000 C CNN
 F 2 "hardwareRev1:SMDJMP-OPEN" H 6700 5450 60  0001 C CNN
@@
 $EndComp
 $Comp
-L SJMPOpen JMP4
+L SJMPOpen JMP101
 U 1 1 55F4BE36
 P 6700 5700
-F 0 "JMP4" H 6900 5850 50  0000 C CNN
+F 0 "JMP101" H 6900 5850 50  0000 C CNN
 F 1 "SJMPOpen" H 6800 5551 40  0000 C CNN
 F 2 "hardwareRev1:SMDJMP-OPEN" H 6700 5700 60  0001 C CNN
@@
 USBV2
 $Comp
-L C C38
+L C C141
 U 1 1 55F4BE38
 P 600 1150
-F 0 "C38" H 600 1250 40  0000 L CNN
+F 0 "C141" H 600 1250 40  0000 L CNN
 F 1 "C" H 606 1065 40  0000 L CNN
 F 2 "Capacitors_SMD:C_0402" H 638 1000 30  0001 C CNN
@@
 internalI2C0SDA
 $Comp
-L CONN_5X2 P4
+L CONN_5X2 P106
 U 1 1 55F4BE3B
 P 5150 2450
-F 0 "P4" H 5150 2750 60  0000 C CNN
+F 0 "P106" H 5150 2750 60  0000 C CNN
 F 1 "CONN_5X2" V 5150 2450 50  0000 C CNN
 F 2 "hardwareRev1:CortexDebug" H 5150 2450 60  0001 C CNN
@@
 $EndComp
 $Comp
-L C C42
+L C C142
 U 1 1 55F4BE45
 P 4750 5600
-F 0 "C42" H 4750 5700 40  0000 L CNN
+F 0 "C142" H 4750 5700 40  0000 L CNN
 F 1 "C" H 4756 5515 40  0000 L CNN
 F 2 "Capacitors_SMD:C_0402" H 4788 5450 30  0001 C CNN
@@
 GPSPulse
 $Comp
-L R R2
+L R R106
 U 1 1 55F4BE54
 P 1050 4000
-F 0 "R2" V 1130 4000 40  0000 C CNN
+F 0 "R106" V 1130 4000 40  0000 C CNN
 F 1 "R" V 1057 4001 40  0000 C CNN
 F 2 "Resistors_SMD:R_0402" V 980 4000 30  0001 C CNN
@@
 $EndComp
 $Comp
-L R R3
+L R R105
 U 1 1 55F4BE55
 P 1250 4000
-F 0 "R3" V 1330 4000 40  0000 C CNN
+F 0 "R105" V 1330 4000 40  0000 C CNN
 F 1 "R" V 1257 4001 40  0000 C CNN
 F 2 "Resistors_SMD:R_0402" V 1180 4000 30  0001 C CNN
@@
 externalSPI1PCS0
 $Comp
-L CONN_8 P3
+L CONN_8 P102
 U 1 1 55F4BE6B
 P 750 7050
-F 0 "P3" V 720 7050 60  0000 C CNN
+F 0 "P102" V 720 7050 60  0000 C CNN
 F 1 "CONN_8" V 820 7050 60  0000 C CNN
 F 2 "Connectors_Molex:Connector_Molex_PicoBlade_53398-0871" H 750 7050 60  0001 C CNN
@@
 LED2
 $Comp
-L R R4
+L R R102
 U 1 1 55F4BE6E
 P 3750 950
-F 0 "R4" V 3830 950 40  0000 C CNN
+F 0 "R102" V 3830 950 40  0000 C CNN
 F 1 "R" V 3757 951 40  0000 C CNN
 F 2 "Resistors_SMD:R_0402" V 3680 950 30  0001 C CNN
@@
 $EndComp
 $Comp
-L R R5
+L R R103
 U 1 1 55F4BE6F
 P 3750 1100
-F 0 "R5" V 3830 1100 40  0000 C CNN
+F 0 "R103" V 3830 1100 40  0000 C CNN
 F 1 "R" V 3757 1101 40  0000 C CNN
 F 2 "Resistors_SMD:R_0402" V 3680 1100 30  0001 C CNN
@@
 $EndComp
 $Comp
-L LED D1
+L LED D101
 U 1 1 55F4BE72
 P 4300 950
-F 0 "D1" H 4300 1050 50  0000 C CNN
+F 0 "D101" H 4300 1050 50  0000 C CNN
 F 1 "LED" H 4300 850 50  0000 C CNN
 F 2 "LEDs:LED-0603" H 4300 950 60  0001 C CNN
@@
 $EndComp
 $Comp
-L LED D2
+L LED D102
 U 1 1 55F4BE73
 P 4300 1100
-F 0 "D2" H 4300 1200 50  0000 C CNN
+F 0 "D102" H 4300 1200 50  0000 C CNN
 F 1 "LED" H 4300 1000 50  0000 C CNN
 F 2 "LEDs:LED-0603" H 4300 1100 60  0001 C CNN
@@
 Connection ~ 7250 5500
 $Comp
-L R R6
+L R R104
 U 1 1 55F4BE75
 P 6000 2950
-F 0 "R6" V 6080 2950 40  0000 C CNN
+F 0 "R104" V 6080 2950 40  0000 C CNN
 F 1 "R" V 6007 2951 40  0000 C CNN
 F 2 "Resistors_SMD:R_0402" V 5930 2950 30  0001 C CNN
@@
 $EndComp
 $Comp
-L CONN_1 P5
+L CONN_1 P105
 U 1 1 55F4BE7D
 P 6350 1600
-F 0 "P5" H 6430 1600 40  0000 L CNN
+F 0 "P105" H 6430 1600 40  0000 L CNN
 F 1 "GPSDM" H 6350 1655 30  0001 C CNN
 F 2 "Measurement_Points:Measurement_Point_Round-SMD-Pad_Small" H 6350 1600 60  0001 C CNN
@@
 $EndComp
 $Comp
-L CONN_1 P6
+L CONN_1 P103
 U 1 1 55F4BE7E
 P 6350 1700
-F 0 "P6" H 6430 1700 40  0000 L CNN
+F 0 "P103" H 6430 1700 40  0000 L CNN
 F 1 "GPSDP" H 6350 1755 30  0001 C CNN
 F 2 "Measurement_Points:Measurement_Point_Round-SMD-Pad_Small" H 6350 1700 60  0001 C CNN
@@
 	7450 5200 7550 5200
 $Comp
-L C C39
+L C C139
 U 1 1 55F4BE80
 P 2350 7400
-F 0 "C39" H 2350 7500 40  0000 L CNN
+F 0 "C139" H 2350 7500 40  0000 L CNN
 F 1 "C" H 2356 7315 40  0000 L CNN
 F 2 "Capacitors_SMD:C_0402" H 2388 7250 30  0001 C CNN
@@
 $EndComp
 $Comp
-L C C40
+L C C140
 U 1 1 55F4BE81
 P 2600 7400
-F 0 "C40" H 2600 7500 40  0000 L CNN
+F 0 "C140" H 2600 7500 40  0000 L CNN
 F 1 "C" H 2606 7315 40  0000 L CNN
 F 2 "Capacitors_SMD:C_0402" H 2638 7250 30  0001 C CNN
@@
 $EndComp
 $Comp
-L C C41
+L C C143
 U 1 1 55F4BE82
 P 2850 7400
-F 0 "C41" H 2850 7500 40  0000 L CNN
+F 0 "C143" H 2850 7500 40  0000 L CNN
 F 1 "C" H 2856 7315 40  0000 L CNN
 F 2 "Capacitors_SMD:C_0402" H 2888 7250 30  0001 C CNN
@@
 Connection ~ 8350 5300
 $Comp
-L C C44
+L C C113
 U 1 1 55F4BE86
 P 9700 1350
-F 0 "C44" H 9700 1450 40  0000 L CNN
+F 0 "C113" H 9700 1450 40  0000 L CNN
 F 1 "C" H 9706 1265 40  0000 L CNN
 F 2 "FC0H224ZFTBR24:FC0H224ZFTBR24" H 9738 1200 30  0001 C CNN
@@
 NoConn ~ 3650 4150
 $Comp
-L MKL26Z128VLH4 U4
+L MKL26Z128VLH4 U105
 U 1 1 55F4BE1B
 P 2700 4050
-F 0 "U4" H 2700 3950 50  0000 C CNN
+F 0 "U105" H 2700 3950 50  0000 C CNN
 F 1 "MKL26Z128VLH4" H 2700 4150 50  0000 C CNN
 F 2 "w_smd_lqfp:lqfp64" H 2700 4050 50  0001 C CNN
@@
 	10850 1050 10850 950
 $Comp
-L INDUCTOR L16
+L INDUCTOR L117
 U 1 1 55F54227
 P 7050 3200
-F 0 "L16" V 7000 3200 40  0000 C CNN
+F 0 "L117" V 7000 3200 40  0000 C CNN
 F 1 "27nH" V 7150 3200 40  0000 C CNN
 F 2 "Resistors_SMD:R_0402" H 7050 3200 60  0001 C CNN
@@
 $EndComp
 $Comp
-L C C43
+L C C144
 U 1 1 55F5430E
 P 6650 3500
-F 0 "C43" H 6650 3600 40  0000 L CNN
+F 0 "C144" H 6650 3600 40  0000 L CNN
 F 1 "47pF" H 6656 3415 40  0000 L CNN
 F 2 "Capacitors_SMD:C_0402" H 6688 3350 30  0001 C CNN
@@
 $EndComp
 $Comp
-L SJMPClosed JMP2
+L SJMPClosed JMP103
 U 1 1 55F545E2
 P 6650 2350
-F 0 "JMP2" H 6850 2500 50  0000 C CNN
+F 0 "JMP103" H 6850 2500 50  0000 C CNN
 F 1 "SJMPClosed" H 6750 2201 40  0000 C CNN
 F 2 "hardwareRev1:SMDJMP-CLOSED" H 6650 2350 60  0001 C CNN
@@
 $EndComp
 $Comp
-L NEO7 RF2
+L NEO7 RF102
 U 1 1 55F548F6
 P 8050 1550
-F 0 "RF2" H 8000 2400 60  0000 C CNN
+F 0 "RF102" H 8000 2400 60  0000 C CNN
 F 1 "NEO7" H 8000 2300 60  0000 C CNN
 F 2 "hardwareRev1:NEO-7" H 8450 1400 60  0001 C CNN
@@
 	9800 1050 8900 1050
 $Comp
-L R R7
+L R R107
 U 1 1 55F555D1
 P 6650 2900
-F 0 "R7" V 6730 2900 40  0000 C CNN
+F 0 "R107" V 6730 2900 40  0000 C CNN
 F 1 "10" V 6657 2901 40  0000 C CNN
 F 2 "Resistors_SMD:R_0402" V 6580 2900 30  0001 C CNN
@@
 $EndComp
 $Comp
-L edgeMountSMA J2
+L edgeMountSMA J102
 U 1 1 55F558F7
 P 7400 2700
-F 0 "J2" H 7525 3015 60  0000 C CNN
+F 0 "J102" H 7525 3015 60  0000 C CNN
 F 1 "edgeMountSMA" H 7590 2940 60  0000 C CNN
 F 2 "hardwareRev1:EdgeSMA" H 7575 2870 50  0000 C CNN
