File: hardware/Radio/radio.sch (KiCad schematic (older format))
At the start: 55 parts, among them J1 edgeMountSMA, J2 edgeMountSMA, P1 CONN_11X2, P2 CONN_1, P3 CONN_8, P4 CONN_5X2, P5 CONN_1, P6 CONN_1, U1 AX503, U2 PE42424, U4 MKL26Z128VLH4, U6 MICRO-B_USB, X1 TCXO

Commit message: Started work on the new power board
Also fixed up some values on the radio board.
Parts:
- C1: value C -> 6.8pf
- C2: value C -> 10pf
- C39, C40, C41, C42: value C -> 1uf
- C5, C6: value C -> 100nf
- L1: value 60nh -> 22nh
- L17: value INDUCTOR -> DNP
- R4, R5: value R -> 80
Changed lines of the file:
@@
 LIBS:RF5110G
 LIBS:PE42424
-LIBS:dra818Real
 LIBS:RFConn
-LIBS:sma
-LIBS:conn_11x2
-LIBS:SparkFun
-LIBS:smtJmpOpen
-LIBS:neo7
-LIBS:MKL26Z128VLH4
-LIBS:USB
-LIBS:open-project
 LIBS:radio-cache
 EELAYER 25 0
@@
 P 3350 4100
 F 0 "C5" H 3350 4200 40  0000 L CNN
-F 1 "C" H 3356 4015 40  0000 L CNN
+F 1 "100nf" H 3356 4015 40  0000 L CNN
 F 2 "Capacitors_SMD:C_0402" H 3388 3950 30  0001 C CNN
 F 3 "" H 3350 4100 60  0000 C CNN
@@
 P 3600 3250
 F 0 "C6" H 3600 3350 40  0000 L CNN
-F 1 "C" H 3606 3165 40  0000 L CNN
+F 1 "100nf" H 3606 3165 40  0000 L CNN
 F 2 "Capacitors_SMD:C_0402" H 3638 3100 30  0001 C CNN
 F 3 "" H 3600 3250 60  0000 C CNN
@@
 P 3150 2950
 F 0 "L1" V 3100 2950 40  0000 C CNN
-F 1 "60nh" V 3250 2950 40  0000 C CNN
+F 1 "22nh" V 3250 2950 40  0000 C CNN
 F 2 "Resistors_SMD:R_0402" H 3150 2950 60  0001 C CNN
 F 3 "" H 3150 2950 60  0000 C CNN
@@
 P 2500 1200
 F 0 "C1" H 2500 1300 40  0000 L CNN
-F 1 "C" H 2506 1115 40  0000 L CNN
+F 1 "6.8pf" H 2506 1115 40  0000 L CNN
 F 2 "Capacitors_SMD:C_0402" H 2538 1050 30  0001 C CNN
 F 3 "" H 2500 1200 60  0000 C CNN
@@
 P 2750 950
 F 0 "C2" H 2750 1050 40  0000 L CNN
-F 1 "C" H 2756 865 40  0000 L CNN
+F 1 "10pf" H 2756 865 40  0000 L CNN
 F 2 "Capacitors_SMD:C_0402" H 2788 800 30  0001 C CNN
 F 3 "" H 2750 950 60  0000 C CNN
@@
 P 2500 -150
 F 0 "C41" H 2500 -50 40  0000 L CNN
-F 1 "C" H 2506 -235 40  0000 L CNN
+F 1 "1uf" H 2506 -235 40  0000 L CNN
 F 2 "Capacitors_SMD:C_0402" H 2538 -300 30  0001 C CNN
 F 3 "" H 2500 -150 60  0000 C CNN
@@
 P 2250 -150
 F 0 "C40" H 2250 -50 40  0000 L CNN
-F 1 "C" H 2256 -235 40  0000 L CNN
+F 1 "1uf" H 2256 -235 40  0000 L CNN
 F 2 "Capacitors_SMD:C_0402" H 2288 -300 30  0001 C CNN
 F 3 "" H 2250 -150 60  0000 C CNN
@@
 P 2000 -150
 F 0 "C39" H 2000 -50 40  0000 L CNN
-F 1 "C" H 2006 -235 40  0000 L CNN
+F 1 "1uf" H 2006 -235 40  0000 L CNN
 F 2 "Capacitors_SMD:C_0402" H 2038 -300 30  0001 C CNN
 F 3 "" H 2000 -150 60  0000 C CNN
@@
 P 3400 -6450
 F 0 "R5" V 3480 -6450 40  0000 C CNN
-F 1 "R" V 3407 -6449 40  0000 C CNN
+F 1 "80" V 3407 -6449 40  0000 C CNN
 F 2 "Resistors_SMD:R_0402" V 3330 -6450 30  0001 C CNN
 F 3 "" H 3400 -6450 30  0000 C CNN
@@
 P 3400 -6600
 F 0 "R4" V 3480 -6600 40  0000 C CNN
-F 1 "R" V 3407 -6599 40  0000 C CNN
+F 1 "80" V 3407 -6599 40  0000 C CNN
 F 2 "Resistors_SMD:R_0402" V 3330 -6600 30  0001 C CNN
 F 3 "" H 3400 -6600 30  0000 C CNN
@@
 P 4400 -1950
 F 0 "C42" H 4400 -1850 40  0000 L CNN
-F 1 "C" H 4406 -2035 40  0000 L CNN
+F 1 "1uf" H 4406 -2035 40  0000 L CNN
 F 2 "Capacitors_SMD:C_0402" H 4438 -2100 30  0001 C CNN
 F 3 "" H 4400 -1950 60  0000 C CNN
@@
 P 5950 3100
 F 0 "L17" V 5900 3100 40  0000 C CNN
-F 1 "INDUCTOR" V 6050 3100 40  0000 C CNN
+F 1 "DNP" V 6050 3100 40  0000 C CNN
 F 2 "Resistors_SMD:R_0402" H 5950 3100 60  0001 C CNN
 F 3 "" H 5950 3100 60  0000 C CNN

Commit message: Really really large commit because I like to live dangerously...
Parts:
- C1, C10, C11, C12, C13, C2, C3, C38, C39, C4, C40, C41, C42, C43, C44, C5, C6, C7, C8, C9: symbol C -> C-RESCUE-radio
- D1, D2: symbol LED -> LED-RESCUE-radio
- R2, R3, R4, R5, R6, R7: symbol R -> R-RESCUE-radio

Commit message: Annotated the schematic and board
Made the numbers increase by 100, so I can just copy this in.
Parts:
- renumbered C4 to C101, C1 to C102, C2 to C103, C9 to C104, C6 to C105, C5 to C106, C7 to C107, C8 to C110, C11 to C111, C10 to C112, C44 to C113, C13 to C115, C12 to C117, C3 to C127, C39 to C139, C40 to C140, C38 to C141, C42 to C142, C41 to C143, C43 to C144, D1 to D101, D2 to D102, J1 to J101, J2 to J102, JMP4 to JMP101, JMP3 to JMP102, JMP2 to JMP103, L1 to L101, L3 to L103, L2 to L104, L5 to L106, L6 to L107, L4 to L108, L17 to L110, L7 to L111, L16 to L117, P1 to P101, P3 to P102, P6 to P103, P2 to P104, P5 to P105, P4 to P106, R4 to R102, R5 to R103, R6 to R104, R3 to R105, R2 to R106, R7 to R107, RF1 to RF101, RF2 to RF102, U1 to U101, U2 to U102, U6 to U104, U4 to U105, X1 to X101
